File: HMI.kicad_sch (KiCad schematic)
At the start: 74 parts, among them J10 S020BQ01HN, J11 Conn_01x02, J12 Molex 104031-0811, M1 C08-005 LRA, 235 Hz, 1.85 V m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, Q3 DMN2075U-7, SW1 RotaryEncoder_Switch, SW2 SW_Push, SW3 SW_Push, SW4 SW_Push, SW5 SW_Push, SW8 SW_Push, U37 SN74AHCT1G125DBVR, U38 DRV2605LDGS, U39 TCA9534PWR, U40 ATECC608C-TCSM, U42 LTR-303ALS-01, U43 PCF85263AT/AJ, Y5 ABS07-32.768KHZ-7-T

Commit message: finished annotation
Parts:
- added R102: 100R, symbol Device:R
- M1: now left out of the parts list
- renumbered C167 to C161, C160 to C162, C159 to C163, C171 to C164, C170 to C165, C175 to C166, C168 to C167, C173 to C168, C174 to C169, C169 to C170, C179 to C171, C180 to C172, C164 to C173, C165 to C174, C172 to C176, C166 to C177, C161 to C179, C177 to C180, C176 to C182, R94 to R100, R95 to R101, R101 to R103, R102 to R104, R100 to R105, R104 to R106, R105 to R107, R106 to R108, R107 to R109, R108 to R110, R109 to R111, R110 to R112, R111 to R113, R88 to R87, R99 to R88, R103 to R89, R97 to R90, R96 to R91, R112 to R92, R113 to R93, R114 to R94, R115 to R95, R116 to R96, R91 to R97, R92 to R98, R93 to R99
Connections:
- net +3V3: now also R102.2; no longer D14.2 (A)
- net SD_DAT2_PU: now reaches J12.1 (DAT2), R92.2
- net BUZZER_DRV: now reaches BZ1.1 (+), R90.1
- net TFT_BL_GATE: now reaches Q3.1 (G), R103.2, R104.2
- net HMI_KEY0_LED_A: now reaches D7.2 (A), R106.1
- net HMI_KEY2_LED_A: now reaches D12.2 (A), R108.1
- net HMI_KEY3_LED_A: now reaches D13.2 (A), R109.1
- net RTC_OSCO: now reaches U43.2 (OSCO), Y5.1
- net RTC_OSCI: now reaches U43.1 (OSCI), Y5.2
- net HMI_KEY1_LED_A: now reaches D11.2 (A), R107.1
- net HAPTIC_REG: now reaches C165.1, U38.1 (REG)
- net HMI_KEY3: now reaches R113.1, SW8.1, U39.7 (P3)
- net WS2812_DATA_5V_RAW: now reaches R91.1, U37.4
- net WS2812_DATA_5V: now reaches D8.4 (DIN), R91.2
- net TFT_BL_K_SW: now reaches Q3.3 (D), R105.1
- net HMI_KEY2: now reaches R112.1, SW5.1, U39.6 (P2)
- net HMI_KEY1: now reaches R111.1, SW4.1, U39.5 (P1)
- net WS2812_CHAIN_2_3: now reaches D10.4 (DIN), D9.2 (DOUT)
- net WS2812_CHAIN_1_2: now reaches D8.2 (DOUT), D9.4 (DIN)
- net ZEROIZE_BTN_RAW: now reaches C177.2, R100.1, R101.1, SW2.1
- net HMI_KEY0: now reaches R110.1, SW3.1, U39.4 (P0)
- net SD_DAT1_PU: now reaches J12.8 (DAT1), R96.2
- net LEDK renamed TFT_BL_K
- net TCA_P4 renamed HMI_KEY_LED_SINK
- new net: D14.2 (A), R102.1
Other:
- note removed: "piezo"
- title: (none) -> Human–Machine Interface, Display, Controls And Storage
- moved on the sheet: BZ1, D11, D12, D13, D14, D7, R106, R107, R108, R109, R88, R91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

Commit message: finished ANCHOR_DOCK sheet
Parts:
- added DS1: S020BQ01HN, symbol Connector_Generic:Conn_01x01
- added J11C1, J11C2: J11 female crimp contact, symbol Connector_Generic:Conn_01x01
- added J11M1: J11 mating housing, 2-position, symbol Connector_Generic:Conn_01x01
- BZ1: DISTRIBUTOR_LINK (none) -> https://www.mouser.com/ProductDetail/Mallory-Sonalert/AST11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; MANUFACTURER (none) -> Mallory Sonalert; MPN (none) -> AST1109MLTRQ; Notes (none) -> N/A
- C161, C162, C166, C167, C168, C169, C171, C176, C177, C178, C180, C182: footprint (none) -> Capacitor_SMD:C_0603_1608Metric; DISTRIBUTOR_LINK (none) -> https://www.mouser.com/ProductDetail/Murata-Electronics/GRM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; MANUFACTURER (none) -> Murata; MPN (none) -> GRM188R71C104KA01D; Notes (none) -> N/A
- C163, C164, C165, C181: footprint (none) -> Capacitor_SMD:C_0603_1608Metric; DISTRIBUTOR_LINK (none) -> https://www.mouser.com/ProductDetail/Murata-Electronics/GRM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; MANUFACTURER (none) -> Murata; MPN (none) -> GRM188R71C105KA12D; Notes (none) -> N/A
- C170, C172: footprint (none) -> Capacitor_SMD:C_0805_2012Metric; DISTRIBUTOR_LINK (none) -> https://www.mouser.com/ProductDetail/Murata-Electronics/GRM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; MANUFACTURER (none) -> Murata; MPN (none) -> GRM21BR71A106KE51L; Notes (none) -> Verify effective capacitance under DC bias.
- C173, C174: footprint (none) -> Capacitor_SMD:C_0603_1608Metric; DISTRIBUTOR_LINK (none) -> https://www.mouser.com/ProductDetail/Murata-Electronics/GRM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; MANUFACTURER (none) -> Murata; MPN (none) -> GRM188R71C103KA01D; Notes (none) -> N/A
- C179: value 11m -> 11mF; DISTRIBUTOR_LINK (none) -> https://www.mouser.com/ProductDetail/Seiko-Semiconductors/C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; MANUFACTURER (none) -> Seiko Instruments; MPN (none) -> CPH3225A; Notes (none) -> Polarized EDLC; preserve pin-1/+ orientation
- D10, D8, D9: DISTRIBUTOR_LINK (none) -> https://www.lcsc.com/product-detail/C114586.html; MANUFACTURER (none) -> Worldsemi; MPN (none) -> WS2812B-B/W; Notes (none) -> PCBWay source exact genuine WS2812B-B/W.
- D11, D12, D13, D7: footprint (none) -> LED_SMD:LED_0603_1608Metric; DISTRIBUTOR_LINK (none) -> https://www.mouser.com/ProductDetail/LITEON/LTST-C190KRKT?q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; MANUFACTURER (none) -> Lite-On; MPN (none) -> LTST-C190KRKT; Notes (none) -> N/A
- D14: DISTRIBUTOR_LINK (none) -> https://www.mouser.com/ProductDetail/Diodes-Incorporated/BA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; MANUFACTURER (none) -> Diodes Incorporated; MPN (none) -> BAV116WS-7; Notes (none) -> N/A
- J10: value S020BQ01HN -> FH12-12S-0.5SH(55); DISTRIBUTOR_LINK (none) -> https://eu.mouser.com/en/ProductDetail/Hirose-Connector/FH1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; MANUFACTURER (none) -> Hirose; MPN (none) -> FH12-12S-0.5SH(55); Notes (none) -> Verified CDTech-recommended connector for S020BQ01HN; botto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
- J11: value Conn_01x02 -> SM02B-GHS-TB(LF)(SN); footprint (none) -> Connector_JST:JST_GH_SM02B-GHS-TB_1x02-1MP_P1.25mm_Horizontal; DISTRIBUTOR_LINK (none) -> https://www.mouser.com/ProductDetail/JST-Commercial/SM02B-G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; MANUFACTURER (none) -> JST; MPN (none) -> SM02B-GHS-TB(LF)(SN); Notes (none) -> Frozen Rev-A pinout: pin 1 HAPTIC_OUT_P/M+, pin 2 HAPTIC_OU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
- J12: DISTRIBUTOR_LINK (none) -> https://www.mouser.com/ProductDetail/Molex/104031-0811?qs=u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; MANUFACTURER (none) -> Molex; MPN (none) -> 104031-0811; Notes (none) -> N/A
- M1: DISTRIBUTOR_LINK (none) -> https://www.precisionmicrodrives.com/products/32931431-4ed1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; MANUFACTURER (none) -> Precision Microdrives; MPN (none) -> C08-005; Notes (none) -> Off-board part connected through J11.; now in the parts list
- Q3: DISTRIBUTOR_LINK (none) -> https://www.mouser.com/ProductDetail/Diodes-Incorporated/DM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; MANUFACTURER (none) -> Diodes Incorporated; MPN (none) -> DMN2075U-7; Notes (none) -> N/A
- R100, R110, R111, R112, R113, R89, R92, R93, R94, R95, R96, R97, R98, R99: footprint (none) -> Resistor_SMD:R_0603_1608Metric; DISTRIBUTOR_LINK (none) -> https://www.mouser.com/ProductDetail/YAGEO/RC0603FR-0710KL?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; MANUFACTURER (none) -> Yageo; MPN (none) -> RC0603FR-0710KL; Notes (none) -> N/A
- R101, R102, R103: footprint (none) -> Resistor_SMD:R_0603_1608Metric; DISTRIBUTOR_LINK (none) -> https://www.mouser.com/ProductDetail/YAGEO/RC0603FR-07100RL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; MANUFACTURER (none) -> Yageo; MPN (none) -> RC0603FR-07100RL; Notes (none) -> N/A
- R104: footprint (none) -> Resistor_SMD:R_0603_1608Metric; DISTRIBUTOR_LINK (none) -> https://www.mouser.com/ProductDetail/YAGEO/RC0603FR-07100KL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; MANUFACTURER (none) -> Yageo; MPN (none) -> RC0603FR-07100KL; Notes (none) -> N/A
- R105: footprint Resistor_SMD:R_1210_3225Metric -> Resistor_SMD:R_1206_3216Metric; DISTRIBUTOR_LINK (none) -> https://www.mouser.com/ProductDetail/Panasonic/ERJ-P08J330V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; MANUFACTURER (none) -> Panasonic; MPN (none) -> ERJ-P08J330V; Notes (none) -> Confirm backlight current and power.
- R106, R107, R108, R109: footprint (none) -> Resistor_SMD:R_0603_1608Metric; DISTRIBUTOR_LINK (none) -> https://www.mouser.com/ProductDetail/YAGEO/RC0603FR-07680RL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; MANUFACTURER (none) -> Yageo; MPN (none) -> RC0603FR-07680RL; Notes (none) -> N/A
- R87, R88: footprint (none) -> Resistor_SMD:R_0603_1608Metric; DISTRIBUTOR_LINK (none) -> https://www.mouser.com/ProductDetail/YAGEO/RC0603FR-072K2L?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; MANUFACTURER (none) -> Yageo; MPN (none) -> RC0603FR-072K2L; Notes (none) -> N/A
- R90: footprint (none) -> Resistor_SMD:R_0603_1608Metric; DISTRIBUTOR_LINK (none) -> https://www.mouser.com/ProductDetail/YAGEO/RC0603FR-07220RL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; MANUFACTURER (none) -> Yageo; MPN (none) -> RC0603FR-07220RL; Notes (none) -> N/A
- R91: footprint (none) -> Resistor_SMD:R_0603_1608Metric; DISTRIBUTOR_LINK (none) -> https://www.mouser.com/ProductDetail/YAGEO/RC0603FR-07330RL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; MANUFACTURER (none) -> Yageo; MPN (none) -> RC0603FR-07330RL; Notes (none) -> N/A
- SW1: DISTRIBUTOR_LINK (none) -> https://www.mouser.com/en/ProductDetail/Bourns/PEC11R-4215F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; MANUFACTURER (none) -> Bourns; MPN (none) -> PEC11R-4215F-S0024; Notes (none) -> Exact Rev-A encoder selected
- SW2, SW3, SW4, SW5, SW8: footprint (none) -> Button_Switch_SMD:SW_SPST_PTS810; DISTRIBUTOR_LINK (none) -> https://eu.mouser.com/en/ProductDetail/CK/PTS810SJM250SMTR-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; MANUFACTURER (none) -> C&K; MPN (none) -> PTS810SJM250SMTR LFS; Notes (none) -> N/A
- U37: DISTRIBUTOR_LINK (none) -> https://www.mouser.com/ProductDetail/Texas-Instruments/SN74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; MANUFACTURER (none) -> Texas Instruments; MPN (none) -> SN74AHCT1G125DBVR; Notes (none) -> N/A
- U38: DISTRIBUTOR_LINK (none) -> https://www.mouser.com/ProductDetail/Texas-Instruments/DRV2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; MANUFACTURER (none) -> Texas Instruments; MPN (none) -> DRV2605LDGSR; Notes (none) -> Configure/calibrate for C08-005.
- U39: DISTRIBUTOR_LINK (none) -> https://www.mouser.com/ProductDetail/Texas-Instruments/TCA9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; MANUFACTURER (none) -> Texas Instruments; MPN (none) -> TCA9534PWR; Notes (none) -> Firmware: I2C address 0x21.
- U40: DISTRIBUTOR_LINK (none) -> https://www.mouser.com/ProductDetail/Microchip-Technology/A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; MANUFACTURER (none) -> Microchip; MPN (none) -> ATECC608C-TCSMS; Notes (none) -> Client approve provisioning before locking.
- U42: DISTRIBUTOR_LINK (none) -> https://www.mouser.com/ProductDetail/LITEON/LTR-303ALS-01?q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; MANUFACTURER (none) -> Lite-On; MPN (none) -> LTR-303ALS-01; Notes (none) -> N/A
- U43: DISTRIBUTOR_LINK (none) -> https://www.mouser.com/ProductDetail/NXP-Semiconductors/PCF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; MANUFACTURER (none) -> NXP; MPN (none) -> PCF85263AT/AJ; Notes (none) -> N/A
- Y5: DISTRIBUTOR_LINK (none) -> https://www.mouser.com/ProductDetail/ABRACON/ABS07-32768KHZ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; MANUFACTURER (none) -> Abracon; MPN (none) -> ABS07-32.768KHZ-7-T; Notes (none) -> N/A
Connections:
- no-connect marks 9 -> 13
Other:
- moved on the sheet: C161

Commit message: the schematic is finished
Other:
- moved on the sheet: BZ1, R90
Changed lines of the file:
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@@
 	(wire
 		(pts
-			(xy 100.33 95.25) (xy 106.68 95.25)
+			(xy 95.25 95.25) (xy 101.6 95.25)
 		)
 		(stroke
@@
 	(wire
 		(pts
-			(xy 114.3 90.17) (xy 129.54 90.17)
+			(xy 109.22 90.17) (xy 124.46 90.17)
 		)
 		(stroke
@@
 	(wire
 		(pts
-			(xy 189.23 114.3) (xy 161.29 114.3)
+			(xy 189.23 115.57) (xy 161.29 115.57)
 		)
 		(stroke
@@
 	(wire
 		(pts
-			(xy 83.82 168.91) (xy 85.09 168.91)
-		)
-		(stroke
-			(width 0)
-			(type default)
-		)
-	)
-	(wire
-		(pts
 			(xy 30.48 27.94) (xy 38.1 27.94)
 		)
@@
 	(wire
 		(pts
-			(xy 100.33 90.17) (xy 100.33 95.25)
+			(xy 95.25 90.17) (xy 95.25 95.25)
 		)
 		(stroke
@@
 	(wire
 		(pts
-			(xy 189.23 110.49) (xy 189.23 114.3)
+			(xy 189.23 110.49) (xy 189.23 115.57)
 		)
 		(stroke
@@
 	(wire
 		(pts
-			(xy 124.46 96.52) (xy 124.46 97.79)
+			(xy 119.38 96.52) (xy 119.38 97.79)
 		)
 		(stroke
@@
 	(wire
 		(pts
-			(xy 129.54 96.52) (xy 129.54 95.25)
+			(xy 124.46 96.52) (xy 124.46 95.25)
 		)
 		(stroke
@@
 	(wire
 		(pts
-			(xy 100.33 90.17) (xy 106.68 90.17)
+			(xy 95.25 90.17) (xy 101.6 90.17)
 		)
 		(stroke
@@
 	(wire
 		(pts
-			(xy 129.54 96.52) (xy 124.46 96.52)
+			(xy 124.46 96.52) (xy 119.38 96.52)
 		)
 		(stroke
@@
 	(wire
 		(pts
+			(xy 161.29 115.57) (xy 161.29 114.3)
+		)
+		(stroke
+			(width 0)
+			(type default)
+		)
+	)
+	(wire
+		(pts
 			(xy 210.82 22.86) (xy 210.82 26.67)
 		)
@@
 	)
 	(label "RTC_OSCO"
-		(at 176.53 114.3 0)
+		(at 176.53 115.57 0)
 		(effects
 			(font
@@
 	)
 	(label "BUZZER_DRV"
-		(at 115.57 90.17 0)
+		(at 110.49 90.17 0)
 		(effects
 			(font
@@
 	)
 	(label "WS2812_DATA_5V"
-		(at 83.82 168.91 180)
+		(at 85.09 168.91 180)
 		(effects
 			(font
@@
 	(hierarchical_label "BUZZER"
 		(shape input)
-		(at 106.68 95.25 0)
+		(at 101.6 95.25 0)
 		(effects
 			(font
@@
 	(symbol
 		(lib_id "Device:Buzzer")
-		(at 132.08 92.71 0)
+		(at 127 92.71 0)
 		(unit 1)
 		(body_style 1)
@@
 		(fields_autoplaced yes)
 		(property "Reference" "BZ1"
-			(at 135.89 91.4399 0)
+			(at 130.81 91.4399 0)
 			(show_name no)
 			(do_not_autoplace no)
@@
 		)
 		(property "Value" "AST1109MLTRQ"
-			(at 135.89 93.9799 0)
+			(at 130.81 93.9799 0)
 			(show_name no)
 			(do_not_autoplace no)
@@
 		)
 		(property "Footprint" "Buzzer_Beeper:Buzzer_Mallory_AST1109MLTRQ"
-			(at 131.445 90.17 90)
+			(at 126.365 90.17 90)
 			(hide yes)
 			(show_name no)
@@
 		)
 		(property "Datasheet" "https://www.mallory-sonalert.com/specifications/AST1109MLTRQ.pdf"
-			(at 131.445 90.17 90)
+			(at 126.365 90.17 90)
 			(hide yes)
 			(show_name no)
@@
 		)
 		(property "Description" "Buzzer, polarized"
-			(at 132.08 92.71 0)
+			(at 127 92.71 0)
 			(hide yes)
 			(show_name no)
@@
 		)
 		(property "DISTRIBUTOR_LINK" "https://www.mouser.com/ProductDetail/Mallory-Sonalert/AST1109MLTRQ?qs=GpRChIzryBM5c7g4uet5pQ%3D%3D"
-			(at 132.08 92.71 0)
+			(at 127 92.71 0)
 			(hide yes)
 			(show_name no)
@@
 		)
 		(property "MPN" "AST1109MLTRQ"
-			(at 132.08 92.71 0)
+			(at 127 92.71 0)
 			(hide yes)
 			(show_name no)
@@
 		)
 		(property "KLC_S3.3" ""
-			(at 132.08 92.71 0)
+			(at 127 92.71 0)
 			(hide yes)
 			(show_name no)
@@
 		)
 		(property "KLC_S4.1" ""
-			(at 132.08 92.71 0)
+			(at 127 92.71 0)
 			(hide yes)
 			(show_name no)
@@
 		)
 		(property "KLC_S4.2_DVDD" ""
-			(at 132.08 92.71 0)
+			(at 127 92.71 0)
 			(hide yes)
 			(show_name no)
@@
 		)
 		(property "KLC_S4.2_VREG_LX" ""
-			(at 132.08 92.71 0)
+			(at 127 92.71 0)
 			(hide yes)
 			(show_name no)
@@
 		)
 		(property "Notes" "N/A"
-			(at 132.08 92.71 0)
+			(at 127 92.71 0)
 			(hide yes)
 			(show_name no)
@@
 		)
 		(property "MANUFACTURER" "Mallory Sonalert"
-			(at 132.08 92.71 0)
+			(at 127 92.71 0)
 			(hide yes)
 			(show_name no)
@@
 		)
 		(property "TUNING_ALTERNATIVES" ""
-			(at 132.08 92.71 0)
+			(at 127 92.71 0)
 			(hide yes)
 			(show_name no)
@@
 	(symbol
 		(lib_id "power:GND")
-		(at 124.46 97.79 0)
+		(at 119.38 97.79 0)
 		(mirror y)
 		(unit 1)
@@
 		(fields_autoplaced yes)
 		(property "Reference" "#PWR0243"
-			(at 124.46 104.14 0)
+			(at 119.38 104.14 0)
 			(hide yes)
 			(show_name no)
@@
 		)
 		(property "Value" "GND"
-			(at 124.46 102.87 0)
+			(at 119.38 102.87 0)
 			(show_name no)
 			(do_not_autoplace no)
@@
 		)
 		(property "Footprint" ""
-			(at 124.46 97.79 0)
+			(at 119.38 97.79 0)
 			(hide yes)
 			(show_name no)
@@
 		)
 		(property "Datasheet" ""
-			(at 124.46 97.79 0)
+			(at 119.38 97.79 0)
 			(hide yes)
 			(show_name no)
@@
 		)
 		(property "Description" "Power symbol creates a global label with name \"GND\" , ground"
-			(at 124.46 97.79 0)
+			(at 119.38 97.79 0)
 			(hide yes)
 			(show_name no)
@@
 	(symbol
 		(lib_id "Device:R")
-		(at 110.49 90.17 270)
+		(at 105.41 90.17 270)
 		(mirror x)
 		(unit 1)
@@
 		(fields_autoplaced yes)
 		(property "Reference" "R90"
-			(at 110.49 83.82 90)
+			(at 105.41 83.82 90)
 			(show_name no)
 			(do_not_autoplace no)
@@
 		)
 		(property "Value" "220R"
-			(at 110.49 86.36 90)
+			(at 105.41 86.36 90)
 			(show_name no)
 			(do_not_autoplace no)
@@
 		)
 		(property "Footprint" "Resistor_SMD:R_0603_1608Metric"
-			(at 110.49 91.948 90)
+			(at 105.41 91.948 90)
 			(hide yes)
 			(show_name no)
@@
 		)
 		(property "Datasheet" "https://www.yageo.com/upload/media/product/productsearch/datasheet/rchip/PYu-RC_Group_51_RoHS_L_11.pdf"
-			(at 110.49 90.17 0)
+			(at 105.41 90.17 0)
 			(hide yes)
 			(show_name no)
@@
 		)
 		(property "Description" "Resistor"
-			(at 110.49 90.17 0)
+			(at 105.41 90.17 0)
 			(hide yes)
 			(show_name yes)
@@
 		)
 		(property "DISTRIBUTOR_LINK" "https://www.mouser.com/ProductDetail/YAGEO/RC0603FR-07220RL?qs=VU8sRB4EgwA1IyQ0vhXEEw%3D%3D"
-			(at 110.49 90.17 90)
+			(at 105.41 90.17 90)
 			(hide yes)
 			(show_name no)
@@
 		)
 		(property "MPN" "RC0603FR-07220RL"
-			(at 110.49 90.17 90)
+			(at 105.41 90.17 90)
 			(hide yes)
 			(show_name no)
@@
 		)
 		(property "KLC_S3.3" ""
-			(at 110.49 90.17 90)
+			(at 105.41 90.17 90)
 			(hide yes)
 			(show_name no)
@@
 		)
 		(property "KLC_S4.1" ""
-			(at 110.49 90.17 90)
+			(at 105.41 90.17 90)
 			(hide yes)
 			(show_name no)
@@
 		)
 		(property "KLC_S4.2_DVDD" ""
-			(at 110.49 90.17 90)
+			(at 105.41 90.17 90)
 			(hide yes)
 			(show_name no)
@@
 		)
 		(property "KLC_S4.2_VREG_LX" ""
-			(at 110.49 90.17 90)
+			(at 105.41 90.17 90)
 			(hide yes)
 			(show_name no)
@@
 		)
 		(property "Notes" "N/A"
-			(at 110.49 90.17 90)
+			(at 105.41 90.17 90)
 			(hide yes)
 			(show_name no)
@@
 		)
 		(property "MANUFACTURER" "Yageo"
-			(at 110.49 90.17 90)
+			(at 105.41 90.17 90)
 			(hide yes)
 			(show_name no)
@@
 		)
 		(property "TUNING_ALTERNATIVES" ""
-			(at 110.49 90.17 90)
+			(at 105.41 90.17 90)
 			(hide yes)
 			(show_name no)

Commit message: finished schematic phase
Parts:
- C179: footprint (none) -> FOBtool_Custom:CP_Seiko_CPH3225A_3.2x2.5mm
- SW1: footprint (none) -> FOBtool_Custom:RotaryEncoder_Bourns_PEC11R-4215F-S0024
Changed lines of the file:
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@@
 			)
 		)
-		(property "Footprint" ""
+		(property "Footprint" "FOBtool_Custom:RotaryEncoder_Bourns_PEC11R-4215F-S0024"
 			(at 177.8 32.766 0)
 			(hide yes)
@@
 			)
 		)
-		(property "Footprint" ""
+		(property "Footprint" "FOBtool_Custom:CP_Seiko_CPH3225A_3.2x2.5mm"
 			(at 228.6 90.4748 0)
 			(hide yes)

Commit message: adding 3d models
Parts:
- J10: symbol Connector_Generic:Conn_01x12 -> FOBtool_Custom:Hirose_FH12_12Pin_MP
- J11: symbol Connector_Generic:Conn_01x02 -> FOBtool_Custom:JST_GH_2Pin_MP
- J12: symbol Connector:Micro_SD_Card_Det1 -> Connector:Micro_SD_Card_Det2
- SW1: symbol Device:RotaryEncoder_Switch -> FOBtool_Custom:Bourns_PEC11R_Switch_MP
Connections:
- no-connect marks 13 -> 17
Changed lines of the file:
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@@
 	)
 	(no_connect
+		(at 49.53 86.36)
+	)
+	(no_connect
 		(at 303.53 185.42)
 	)
 	(no_connect
+		(at 68.58 228.6)
+	)
+	(no_connect
 		(at 68.58 231.14)
 	)
@@
 	)
 	(no_connect
+		(at 41.91 57.15)
+	)
+	(no_connect
 		(at 303.53 190.5)
 	)
 	(no_connect
+		(at 189.23 43.18)
+	)
+	(no_connect
 		(at 52.07 31.75)
 	)
@@
 	)
 	(symbol
-		(lib_id "Device:RotaryEncoder_Switch")
+		(lib_id "FOBtool_Custom:Bourns_PEC11R_Switch_MP")
 		(at 181.61 36.83 0)
 		(unit 1)
@@
 		(pin "A"
 		)
+		(pin "MP"
+		)
 		(instances
 			(project "FOBtool_HW"
@@
 	)
 	(symbol
-		(lib_id "Connector_Generic:Conn_01x02")
+		(lib_id "FOBtool_Custom:JST_GH_2Pin_MP")
 		(at 44.45 83.82 0)
 		(unit 1)
@@
 		(fields_autoplaced yes)
 		(property "Reference" "J11"
-			(at 46.99 83.8199 0)
+			(at 44.45 77.47 0)
 			(show_name no)
 			(do_not_autoplace no)
@@
 					(size 1.27 1.27)
 				)
-				(justify left)
 			)
 		)
 		(property "Value" "SM02B-GHS-TB(LF)(SN)"
-			(at 46.99 86.3599 0)
+			(at 44.45 80.01 0)
 			(show_name no)
 			(do_not_autoplace no)
@@
 					(size 1.27 1.27)
 				)
-				(justify left)
 			)
 		)
@@
 		(pin "2"
 		)
+		(pin "MP"
+		)
 		(instances
 			(project "FOBtool_HW"
@@
 	)
 	(symbol
-		(lib_id "Connector_Generic:Conn_01x12")
+		(lib_id "FOBtool_Custom:Hirose_FH12_12Pin_MP")
 		(at 46.99 41.91 0)
 		(mirror y)
@@
 		(pin "12"
 		)
+		(pin "MP"
+		)
 		(instances
 			(project "FOBtool_HW"
@@
 		(in_pos_files yes)
 		(dnp no)
-		(fields_autoplaced yes)
 		(property "Reference" "#PWR0221"
 			(at 215.9 21.59 0)
@@
 		)
 		(property "Value" "+3V3"
-			(at 215.9 12.7 0)
+			(at 220.218 15.24 0)
 			(show_name no)
 			(do_not_autoplace no)
@@
 	)
 	(symbol
-		(lib_id "Connector:Micro_SD_Card_Det1")
+		(lib_id "Connector:Micro_SD_Card_Det2")
 		(at 45.72 218.44 0)
 		(mirror y)
@@
 			)
 		)
-		(property "Datasheet" "https://www.molex.com/en-us/products/part-detail/1040310811"
-			(at 45.72 215.9 0)
+		(property "Datasheet" "https://www.hirose.com/en/product/document?clcode=&productname=&series=DM3&documenttype=Catalog&lang=en&documentid=D49662_en"
+			(at 43.18 215.9 0)
 			(hide yes)
 			(show_name no)
@@
 			)
 		)
-		(property "Description" "Micro SD Card Socket with one card detection pin"
+		(property "Description" "Micro SD Card Socket with two card detection pins"
 			(at 45.72 218.44 0)
 			(hide yes)
@@
 			)
 		)
-		(pin "SH"
-		)
-		(pin "9"
-		)
 		(pin "1"
 		)
 		(pin "6"
 		)
-		(pin "7"
-		)
-		(pin "8"
-		)
 		(pin "5"
 		)
@@
 		(pin "2"
 		)
+		(pin "9"
+		)
+		(pin "10"
+		)
+		(pin "8"
+		)
+		(pin "7"
+		)
+		(pin "SH"
+		)
 		(instances
