File: FOBtool_HW.kicad_pcb (KiCad board)
At the start: 6 copper layers, 0 parts

Commit message: adding 3d models
Parts:
- added AE1: UWA.01, FOBtool_Custom:Antenna_Taoglas_UWA01_3.2x1.6mm, F.Cu at (77.3, 132.5)
- added AE2: UWA.01, FOBtool_Custom:Antenna_Taoglas_UWA01_3.2x1.6mm, F.Cu at (77.3, 139.6)
- added BZ1: AST1109MLTRQ, Buzzer_Beeper:Buzzer_Mallory_AST1109MLTRQ, F.Cu at (136.4, 55.9)
- added C1: 1u, Capacitor_SMD:C_0603_1608Metric, F.Cu at (140.7, 129.1)
- added C10: 47u, Capacitor_SMD:C_1210_3225Metric, F.Cu at (164.6, 138.5)
- added C100: 2u2, Capacitor_SMD:C_0603_1608Metric, F.Cu at (62.8, 39.3)
- added C101: 1n, Capacitor_SMD:C_0402_1005Metric, F.Cu at (73.7, 56.1)
- added C102: 10u, Capacitor_SMD:C_0805_2012Metric, F.Cu at (69.6, 98.4)
- added C103: 100n, Capacitor_SMD:C_0402_1005Metric, F.Cu at (73.7, 58.0)
- added C104: 100n, Capacitor_SMD:C_0402_1005Metric, F.Cu at (73.7, 60.0)
- added C105: 100n, Capacitor_SMD:C_0402_1005Metric, F.Cu at (73.7, 62.0)
- added C106: 100n, Capacitor_SMD:C_0402_1005Metric, F.Cu at (73.7, 63.9)
- added C107: 100n, Capacitor_SMD:C_0402_1005Metric, F.Cu at (73.7, 65.9)
- added C108: 100n, Capacitor_SMD:C_0402_1005Metric, F.Cu at (73.7, 67.9)
- added C109: NM, Capacitor_SMD:C_0402_1005Metric, F.Cu at (73.7, 69.8)
- added C11: 22u, Capacitor_SMD:C_1206_3216Metric, F.Cu at (135.8, 139.6)
- added C110: 1p2, Capacitor_SMD:C_0402_1005Metric, F.Cu at (73.7, 71.8)
- added C111: 1u, Capacitor_SMD:C_0603_1608Metric, F.Cu at (62.8, 41.8)
- added C112: 100n, Capacitor_SMD:C_0402_1005Metric, F.Cu at (73.7, 73.8)
- added C113: 100p, Capacitor_SMD:C_0402_1005Metric, F.Cu at (73.7, 75.8)
- added C114: 0p6, Capacitor_SMD:C_0402_1005Metric, F.Cu at (73.7, 77.7)
- added C115: 100p, Capacitor_SMD:C_0402_1005Metric, F.Cu at (76.5, 54.1)
- added C116: 15p, Capacitor_SMD:C_0402_1005Metric, F.Cu at (76.5, 56.1)
- added C117: 15p, Capacitor_SMD:C_0402_1005Metric, F.Cu at (76.5, 58.0)
- added C118: 100n, Capacitor_SMD:C_0402_1005Metric, F.Cu at (76.5, 60.0)
- added C119: 100n, Capacitor_SMD:C_0402_1005Metric, F.Cu at (76.5, 62.0)
- added C12: 22u, Capacitor_SMD:C_1206_3216Metric, F.Cu at (135.8, 142.9)
- added C120: 100p, Capacitor_SMD:C_0402_1005Metric, F.Cu at (76.5, 63.9)
- added C121: 100n, Capacitor_SMD:C_0402_1005Metric, F.Cu at (76.5, 65.9)
- added C122: 100p, Capacitor_SMD:C_0402_1005Metric, F.Cu at (76.5, 67.9)
- added C123: 100p, Capacitor_SMD:C_0402_1005Metric, F.Cu at (76.5, 69.8)
- added C124: 1u, Capacitor_SMD:C_0603_1608Metric, F.Cu at (62.8, 44.3)
- added C125: 100p, Capacitor_SMD:C_0402_1005Metric, F.Cu at (76.5, 71.8)
- added C126: 100n, Capacitor_SMD:C_0402_1005Metric, F.Cu at (76.5, 73.8)
- added C127: 100n, Capacitor_SMD:C_0402_1005Metric, F.Cu at (76.5, 75.8)
- added C128: 100n, Capacitor_SMD:C_0402_1005Metric, F.Cu at (76.5, 77.7)
- added C129: 100n, Capacitor_SMD:C_0402_1005Metric, F.Cu at (79.4, 54.1)
- added C13: 2u2, Capacitor_SMD:C_0603_1608Metric, F.Cu at (140.7, 134.1)
- added C130: 100n, Capacitor_SMD:C_0402_1005Metric, F.Cu at (79.4, 56.1)
- added C131: 100n, Capacitor_SMD:C_0402_1005Metric, F.Cu at (79.4, 58.0)
- added C132: 1u, Capacitor_SMD:C_0603_1608Metric, F.Cu at (62.8, 46.8)
- added C134: 100n, Capacitor_SMD:C_0402_1005Metric, F.Cu at (79.4, 60.0)
- added C135: 15p, Capacitor_SMD:C_0402_1005Metric, F.Cu at (79.4, 62.0)
- added C136: 15p, Capacitor_SMD:C_0402_1005Metric, F.Cu at (79.4, 63.9)
- added C137: 100n, Capacitor_SMD:C_0402_1005Metric, F.Cu at (79.4, 65.9)
- added C138: 100p, Capacitor_SMD:C_0402_1005Metric, F.Cu at (79.4, 67.9)
- added C139: 100p, Capacitor_SMD:C_0402_1005Metric, F.Cu at (79.4, 69.8)
- added C14: 10p, Capacitor_SMD:C_0603_1608Metric, F.Cu at (140.7, 136.7)
- added C140: 0p6, Capacitor_SMD:C_0402_1005Metric, F.Cu at (79.4, 71.8)
- added C141: 100p, Capacitor_SMD:C_0402_1005Metric, F.Cu at (79.4, 73.8)
- added C142: 100p, Capacitor_SMD:C_0402_1005Metric, F.Cu at (79.4, 75.8)
- added C143: 1u, Capacitor_SMD:C_0603_1608Metric, F.Cu at (62.8, 49.3)
- added C144: 100p, Capacitor_SMD:C_0402_1005Metric, F.Cu at (79.4, 77.7)
- added C145: NM, Capacitor_SMD:C_0402_1005Metric, F.Cu at (82.3, 54.1)
- added C146: 1p2, Capacitor_SMD:C_0402_1005Metric, F.Cu at (82.3, 56.1)
- added C147: 100n, Capacitor_SMD:C_0402_1005Metric, F.Cu at (82.3, 58.0)
- added C148: 100n, Capacitor_SMD:C_0402_1005Metric, F.Cu at (82.3, 60.0)
- added C149: 100n, Capacitor_SMD:C_0402_1005Metric, F.Cu at (82.3, 62.0)
- added C15: 1n, Capacitor_SMD:C_0603_1608Metric, F.Cu at (140.7, 139.2)
- added C150: 100n, Capacitor_SMD:C_0603_1608Metric, F.Cu at (100.4, 146.4)
- added C151: 100p, Capacitor_SMD:C_0603_1608Metric, F.Cu at (100.4, 148.9)
- added C152: 100p, Capacitor_SMD:C_0603_1608Metric, F.Cu at (100.4, 151.5)
- added C153: 4u7, Capacitor_SMD:C_0603_1608Metric, F.Cu at (100.4, 154.0)
- added C154: 100n, Capacitor_SMD:C_0603_1608Metric, F.Cu at (100.4, 156.5)
- added C155: 4u7, Capacitor_SMD:C_0603_1608Metric, F.Cu at (100.4, 159.0)
- added C156: 100n, Capacitor_SMD:C_0603_1608Metric, F.Cu at (104.4, 146.4)
- added C157: 10u, Capacitor_SMD:C_0805_2012Metric, F.Cu at (123.7, 142.2)
- added C158: 100n, Capacitor_SMD:C_0603_1608Metric, F.Cu at (104.4, 148.9)
- added C159: 100n, Capacitor_SMD:C_0603_1608Metric, F.Cu at (104.4, 151.5)
- added C16: 100n, Capacitor_SMD:C_0603_1608Metric, F.Cu at (140.7, 141.7)
- added C160: 4n7, Capacitor_SMD:C_0603_1608Metric, F.Cu at (104.4, 154.0)
- added C161: 100n, Capacitor_SMD:C_0603_1608Metric, F.Cu at (100.4, 29.3)
- added C162: 100n, Capacitor_SMD:C_0603_1608Metric, F.Cu at (100.4, 31.8)
- added C163: 1u, Capacitor_SMD:C_0603_1608Metric, F.Cu at (100.4, 34.3)
- added C164: 1u, Capacitor_SMD:C_0603_1608Metric, F.Cu at (100.4, 36.8)
- added C165: 1u, Capacitor_SMD:C_0603_1608Metric, F.Cu at (100.4, 39.3)
- added C166: 100n, Capacitor_SMD:C_0603_1608Metric, F.Cu at (100.4, 41.8)
- added C167: 100n, Capacitor_SMD:C_0603_1608Metric, F.Cu at (100.4, 44.3)
- added C168: 100n, Capacitor_SMD:C_0603_1608Metric, F.Cu at (100.4, 46.8)
- added C169: 100n, Capacitor_SMD:C_0603_1608Metric, F.Cu at (100.4, 49.3)
- added C17: 0u1, Capacitor_SMD:C_0603_1608Metric, F.Cu at (144.7, 129.1)
- added C170: 10u, Capacitor_SMD:C_0805_2012Metric, F.Cu at (139.3, 71.6)
- added C171: 100n, Capacitor_SMD:C_0603_1608Metric, F.Cu at (104.4, 29.3)
- added C172: 10u, Capacitor_SMD:C_0805_2012Metric, F.Cu at (139.3, 74.6)
- added C173: 10n, Capacitor_SMD:C_0603_1608Metric, F.Cu at (104.4, 31.8)
- added C174: 10n, Capacitor_SMD:C_0603_1608Metric, F.Cu at (104.4, 34.3)
- added C176: 100n, Capacitor_SMD:C_0603_1608Metric, F.Cu at (104.4, 36.8)
- added C177: 100n, Capacitor_SMD:C_0603_1608Metric, F.Cu at (104.4, 39.3)
- added C178: 100n, Capacitor_SMD:C_0603_1608Metric, F.Cu at (104.4, 41.8)
- added C179: 11mF, FOBtool_Custom:CP_Seiko_CPH3225A_3.2x2.5mm, F.Cu at (122.6, 72.5)
- added C18: 120u, FOBtool_Custom:CP_Panasonic_EEF-TX_7.3x4.3mm, F.Cu at (161.7, 152.2)
- added C180: 100n, Capacitor_SMD:C_0603_1608Metric, F.Cu at (104.4, 44.3)
- added C181: 1u, Capacitor_SMD:C_0603_1608Metric, F.Cu at (104.4, 46.8)
- added C182: 100n, Capacitor_SMD:C_0603_1608Metric, F.Cu at (104.4, 49.3)
- added C183: 220n, Capacitor_SMD:C_0402_1005Metric, F.Cu at (82.8, 131.9)
- added C184: 100n, Capacitor_SMD:C_0402_1005Metric, F.Cu at (82.8, 133.8)
- added C185: 4n7, Capacitor_SMD:C_0402_1005Metric, F.Cu at (82.8, 135.8)
- added C186: 10u, Capacitor_SMD:C_0805_2012Metric, F.Cu at (43.7, 132.4)
- added C187: 100n, Capacitor_SMD:C_0402_1005Metric, F.Cu at (82.8, 137.8)
- added C188: 4n7, Capacitor_SMD:C_0402_1005Metric, F.Cu at (82.8, 139.7)
- added C189: 10u, Capacitor_SMD:C_0805_2012Metric, F.Cu at (43.7, 135.4)
- added C19: 22u, Capacitor_SMD:C_1206_3216Metric, F.Cu at (135.8, 146.3)
- added C190: 10u, Capacitor_SMD:C_0805_2012Metric, F.Cu at (43.7, 138.4)
- added C191: 4n7, Capacitor_SMD:C_0402_1005Metric, F.Cu at (82.8, 141.7)
- added C192: 100n, Capacitor_SMD:C_0402_1005Metric, F.Cu at (82.8, 143.7)
- added C193: 22u, Capacitor_SMD:C_1206_3216Metric, F.Cu at (70.1, 132.5)
- added C194: 2p, Capacitor_SMD:C_0402_1005Metric, F.Cu at (85.7, 131.9)
- added C195: 100n, Capacitor_SMD:C_0402_1005Metric, F.Cu at (85.7, 133.8)
- added C196: 100n, Capacitor_SMD:C_0402_1005Metric, F.Cu at (85.7, 135.8)
- added C197: 2p, Capacitor_SMD:C_0402_1005Metric, F.Cu at (85.7, 137.8)
- added C198: NM, Capacitor_SMD:C_0402_1005Metric, F.Cu at (85.7, 139.7)
- added C199: 2p, Capacitor_SMD:C_0402_1005Metric, F.Cu at (85.7, 141.7)
- added C2: 22u, Capacitor_SMD:C_1206_3216Metric, F.Cu at (135.8, 129.5)
- added C20: 22u, Capacitor_SMD:C_1206_3216Metric, F.Cu at (135.8, 149.6)
- added C200: NM, Capacitor_SMD:C_0402_1005Metric, F.Cu at (85.7, 143.7)
- added C201: 2p, Capacitor_SMD:C_0402_1005Metric, F.Cu at (88.6, 131.9)
- added C202: 2p, Capacitor_SMD:C_0402_1005Metric, F.Cu at (88.6, 133.8)
- added C203: 100n, Capacitor_SMD:C_0402_1005Metric, F.Cu at (88.6, 135.8)
- added C204: 10u, Capacitor_SMD:C_0805_2012Metric, F.Cu at (43.7, 141.4)
- added C205: 10n, Capacitor_SMD:C_0603_1608Metric, F.Cu at (43.5, 104.5)
- added C206: 100n, Capacitor_SMD:C_0603_1608Metric, F.Cu at (43.5, 107.0)
- added C207: 100n, Capacitor_SMD:C_0603_1608Metric, F.Cu at (43.5, 109.5)
- added C208: 1n, Capacitor_SMD:C_0603_1608Metric, F.Cu at (43.5, 112.0)
- added C209: 100n, Capacitor_SMD:C_0603_1608Metric, F.Cu at (43.5, 114.6)
- added C21: 22u, Capacitor_SMD:C_1206_3216Metric, F.Cu at (135.8, 153.0)
- added C210: 100n, Capacitor_SMD:C_0603_1608Metric, F.Cu at (43.5, 117.1)
- added C211: 22u, Capacitor_SMD:C_1206_3216Metric, F.Cu at (70.1, 135.9)
- added C212: 22u, Capacitor_SMD:C_1206_3216Metric, F.Cu at (70.1, 139.2)
- added C213: 47p, Capacitor_SMD:C_0603_1608Metric, F.Cu at (43.5, 119.6)
- added C214: 100p, Capacitor_SMD:C_0603_1608Metric, F.Cu at (43.5, 122.1)
- added C215: 220p, Capacitor_SMD:C_0603_1608Metric, F.Cu at (43.5, 124.6)
- added C216: 220p, Capacitor_SMD:C_0603_1608Metric, F.Cu at (43.5, 127.1)
- added C217: 3n3, Capacitor_SMD:C_0603_1608Metric, F.Cu at (43.5, 129.6)
- added C218: 220p, Capacitor_SMD:C_0603_1608Metric, F.Cu at (47.5, 104.5)
- added C219: 100n, Capacitor_SMD:C_0603_1608Metric, F.Cu at (47.5, 107.0)
- added C22: 10u, Capacitor_SMD:C_0805_2012Metric, F.Cu at (146.5, 161.7)
- added C220: 100n, Capacitor_SMD:C_0603_1608Metric, F.Cu at (47.5, 109.5)
- added C221: 22u, Capacitor_SMD:C_1206_3216Metric, F.Cu at (70.1, 142.6)
- added C222: 22u, Capacitor_SMD:C_1206_3216Metric, F.Cu at (70.1, 145.9)
- added C223: 47p, Capacitor_SMD:C_0603_1608Metric, F.Cu at (47.5, 112.0)
- added C224: 100p, Capacitor_SMD:C_0603_1608Metric, F.Cu at (47.5, 114.6)
- added C225: 220p, Capacitor_SMD:C_0603_1608Metric, F.Cu at (47.5, 117.1)
- added C226: 1n, Capacitor_SMD:C_0603_1608Metric, F.Cu at (47.5, 119.6)
- added C227: 220p, Capacitor_SMD:C_0603_1608Metric, F.Cu at (47.5, 122.1)
- added C228: 3n3, Capacitor_SMD:C_0603_1608Metric, F.Cu at (47.5, 124.6)
- added C229: 220p, Capacitor_SMD:C_0603_1608Metric, F.Cu at (47.5, 127.1)
- added C23: 1u, Capacitor_SMD:C_0603_1608Metric, F.Cu at (149.4, 81.5)
- added C230: 1u, Capacitor_SMD:C_0603_1608Metric, F.Cu at (47.5, 129.6)
- added C231: 4u7, Capacitor_SMD:C_0805_2012Metric, F.Cu at (43.7, 144.4)
- added C232: 100n, Capacitor_SMD:C_0603_1608Metric, F.Cu at (51.5, 104.5)
- added C233: 2u2, Capacitor_SMD:C_0603_1608Metric, F.Cu at (51.5, 107.0)
- added C234: 2u2, Capacitor_SMD:C_0603_1608Metric, F.Cu at (51.5, 109.5)
- added C235: 12p, Capacitor_SMD:C_0603_1608Metric, F.Cu at (51.5, 112.0)
- added C236: 12p, Capacitor_SMD:C_0603_1608Metric, F.Cu at (51.5, 114.6)
- added C237: 100n, Capacitor_SMD:C_0603_1608Metric, F.Cu at (51.5, 117.1)
- added C238: 4u7, Capacitor_SMD:C_0805_2012Metric, F.Cu at (43.7, 147.4)
- added C239: 330p, Capacitor_SMD:C_0603_1608Metric, F.Cu at (51.5, 119.6)
- added C24: 22u, Capacitor_SMD:C_1206_3216Metric, F.Cu at (101.2, 124.2)
- added C240: NM, Capacitor_SMD:C_0603_1608Metric, F.Cu at (51.5, 122.1)
- added C241: 68p, Capacitor_SMD:C_0603_1608Metric, F.Cu at (51.5, 124.6)
- added C242: NM, Capacitor_SMD:C_0603_1608Metric, F.Cu at (51.5, 127.1)
- added C243: 100p, Capacitor_SMD:C_0603_1608Metric, F.Cu at (51.5, 129.6)
- added C244: NM, Capacitor_SMD:C_0603_1608Metric, F.Cu at (55.5, 104.5)
- added C245: 330p, Capacitor_SMD:C_0603_1608Metric, F.Cu at (55.5, 107.0)
- added C246: NM, Capacitor_SMD:C_0603_1608Metric, F.Cu at (55.5, 109.5)
- added C247: 68p, Capacitor_SMD:C_0603_1608Metric, F.Cu at (55.5, 112.0)
- added C248: NM, Capacitor_SMD:C_0603_1608Metric, F.Cu at (55.5, 114.6)
- added C249: 100p, Capacitor_SMD:C_0603_1608Metric, F.Cu at (55.5, 117.1)
- added C25: 100n, Capacitor_SMD:C_0603_1608Metric, F.Cu at (149.4, 84.0)
- added C250: NM, Capacitor_SMD:C_0603_1608Metric, F.Cu at (55.5, 119.6)
- added C251: 1n, Capacitor_SMD:C_0603_1608Metric, F.Cu at (55.5, 122.1)
- added C252: 1n, Capacitor_SMD:C_0603_1608Metric, F.Cu at (55.5, 124.6)
- added C253: 15p, Capacitor_SMD:C_0603_1608Metric, F.Cu at (55.5, 127.1)
- added C254: 15p, Capacitor_SMD:C_0603_1608Metric, F.Cu at (55.5, 129.6)
- added C255: 2u2, Capacitor_SMD:C_0603_1608Metric, F.Cu at (59.5, 104.5)
- added C256: 2u2, Capacitor_SMD:C_0603_1608Metric, F.Cu at (59.5, 107.0)
- added C257: DNP, Capacitor_SMD:C_0402_1005Metric, F.Cu at (88.6, 137.8)
- added C258: DNP, Capacitor_SMD:C_0402_1005Metric, F.Cu at (88.6, 139.7)
- added C259: 100n, Capacitor_SMD:C_0603_1608Metric, F.Cu at (148.9, 55.8)
- added C26: 4u7, Capacitor_SMD:C_0603_1608Metric, F.Cu at (148.9, 29.3)
- added C260: 100n, Capacitor_SMD:C_0603_1608Metric, F.Cu at (148.9, 58.3)
- added C261: 22u, Capacitor_SMD:C_1206_3216Metric, F.Cu at (155.6, 68.8)
- added C262: 100n, Capacitor_SMD:C_0603_1608Metric, F.Cu at (148.9, 60.8)
- added C27: 100n, Capacitor_SMD:C_0402_1005Metric, F.Cu at (156.4, 45.2)
- added C28: 100n, Capacitor_SMD:C_0402_1005Metric, F.Cu at (156.4, 47.2)
- added C29: 4u7, Capacitor_SMD:C_0603_1608Metric, F.Cu at (148.9, 31.8)
- added C3: 47n, Capacitor_SMD:C_0603_1608Metric, F.Cu at (140.7, 131.6)
- added C30: 15p, Capacitor_SMD:C_0402_1005Metric, F.Cu at (156.4, 49.1)
- added C31: 15p, Capacitor_SMD:C_0402_1005Metric, F.Cu at (156.4, 51.1)
- added C32: 4u7, Capacitor_SMD:C_0603_1608Metric, F.Cu at (148.9, 34.3)
- added C33: 100n, Capacitor_SMD:C_0402_1005Metric, F.Cu at (159.2, 45.2)
- added C34: 100n, Capacitor_SMD:C_0402_1005Metric, F.Cu at (159.2, 47.2)
- added C35: 100n, Capacitor_SMD:C_0402_1005Metric, F.Cu at (159.2, 49.1)
- added C36: 100n, Capacitor_SMD:C_0402_1005Metric, F.Cu at (159.2, 51.1)
- added C37: 100n, Capacitor_SMD:C_0402_1005Metric, F.Cu at (162.1, 45.2)
- added C38: 100n, Capacitor_SMD:C_0402_1005Metric, F.Cu at (162.1, 47.2)
- added C39: 100n, Capacitor_SMD:C_0402_1005Metric, F.Cu at (162.1, 49.1)
- added C4: 22u, Capacitor_SMD:C_1206_3216Metric, F.Cu at (135.8, 132.9)
- added C40: 10u, Capacitor_SMD:C_0805_2012Metric, F.Cu at (167.5, 29.5)
- added C41: 100n, Capacitor_SMD:C_0402_1005Metric, F.Cu at (162.1, 51.1)
- added C42: 100n, Capacitor_SMD:C_0402_1005Metric, F.Cu at (62.2, 54.1)
- added C43: 4p7, Capacitor_SMD:C_0402_1005Metric, F.Cu at (62.2, 56.1)
- added C44: 4p7, Capacitor_SMD:C_0402_1005Metric, F.Cu at (62.2, 58.0)
- added C45: 1u, Capacitor_SMD:C_0603_1608Metric, F.Cu at (62.8, 29.3)
- added C46: 100n, Capacitor_SMD:C_0402_1005Metric, F.Cu at (62.2, 60.0)
- added C47: 100n, Capacitor_SMD:C_0402_1005Metric, F.Cu at (62.2, 62.0)
- added C48: 1p, Capacitor_SMD:C_0402_1005Metric, F.Cu at (62.2, 63.9)
- added C49: 3p, Capacitor_SMD:C_0402_1005Metric, F.Cu at (62.2, 65.9)
- added C5: 22u, Capacitor_SMD:C_1206_3216Metric, F.Cu at (135.8, 136.2)
- added C50: 3p9, Capacitor_SMD:C_0402_1005Metric, F.Cu at (62.2, 67.9)
- added C51: 5p1, Capacitor_SMD:C_0402_1005Metric, F.Cu at (62.2, 69.8)
- added C52: 2p7, Capacitor_SMD:C_0402_1005Metric, F.Cu at (62.2, 71.8)
- added C53: 100p, Capacitor_SMD:C_0402_1005Metric, F.Cu at (62.2, 73.8)
- added C54: 100p, Capacitor_SMD:C_0402_1005Metric, F.Cu at (62.2, 75.8)
- added C55: 8p2, Capacitor_SMD:C_0402_1005Metric, F.Cu at (62.2, 77.7)
- added C56: 15p, Capacitor_SMD:C_0402_1005Metric, F.Cu at (65.1, 54.1)
- added C57: 100p, Capacitor_SMD:C_0402_1005Metric, F.Cu at (65.1, 56.1)
- added C58: 1u, Capacitor_SMD:C_0603_1608Metric, F.Cu at (62.8, 31.8)
- added C59: 100p, Capacitor_SMD:C_0402_1005Metric, F.Cu at (65.1, 58.0)
- added C6: 10u, Capacitor_SMD:C_0805_2012Metric, F.Cu at (146.5, 155.7)
- added C60: 68u, FOBtool_Custom:CP_Panasonic_EEF-LR_7.3x4.3mm_3Terminal, F.Cu at (83.7, 96.0)
- added C61: 1000p, Capacitor_SMD:C_0402_1005Metric, F.Cu at (65.1, 60.0)
- added C62: 100p, Capacitor_SMD:C_0402_1005Metric, F.Cu at (65.1, 62.0)
- added C63: 1000p, Capacitor_SMD:C_0402_1005Metric, F.Cu at (65.1, 63.9)
- added C64: 22p, Capacitor_SMD:C_0402_1005Metric, F.Cu at (65.1, 65.9)
- added C65: 22p, Capacitor_SMD:C_0402_1005Metric, F.Cu at (65.1, 67.9)
- added C66: 6p8, Capacitor_SMD:C_0402_1005Metric, F.Cu at (65.1, 69.8)
- added C67: 4p7, Capacitor_SMD:C_0402_1005Metric, F.Cu at (65.1, 71.8)
- added C68: 15p, Capacitor_SMD:C_0402_1005Metric, F.Cu at (65.1, 73.8)
- added C69: 13p, Capacitor_SMD:C_0402_1005Metric, F.Cu at (65.1, 75.8)
- added C7: 4u7, Capacitor_SMD:C_0805_2012Metric, F.Cu at (146.5, 158.7)
- added C70: 3p3, Capacitor_SMD:C_0402_1005Metric, F.Cu at (65.1, 77.7)
- added C71: 11p, Capacitor_SMD:C_0402_1005Metric, F.Cu at (67.9, 54.1)
- added C72: 9p1, Capacitor_SMD:C_0402_1005Metric, F.Cu at (67.9, 56.1)
- added C73: 1p8, Capacitor_SMD:C_0402_1005Metric, F.Cu at (67.9, 58.0)
- added C74: 5p6, Capacitor_SMD:C_0402_1005Metric, F.Cu at (67.9, 60.0)
- added C75: 4p7, Capacitor_SMD:C_0402_1005Metric, F.Cu at (67.9, 62.0)
- added C76: 100p, Capacitor_SMD:C_0402_1005Metric, F.Cu at (67.9, 63.9)
- added C77: 100p, Capacitor_SMD:C_0402_1005Metric, F.Cu at (67.9, 65.9)
- added C78: 0p6, Capacitor_SMD:C_0402_1005Metric, F.Cu at (67.9, 67.9)
- added C79: 1u, Capacitor_SMD:C_0603_1608Metric, F.Cu at (62.8, 34.3)
- added C8: 47u, Capacitor_SMD:C_1210_3225Metric, F.Cu at (164.6, 130.0)
- added C80: 100n, Capacitor_SMD:C_0402_1005Metric, F.Cu at (67.9, 69.8)
- added C81: 15p, Capacitor_SMD:C_0402_1005Metric, F.Cu at (67.9, 71.8)
- added C82: 15p, Capacitor_SMD:C_0402_1005Metric, F.Cu at (67.9, 73.8)
- added C83: 100n, Capacitor_SMD:C_0402_1005Metric, F.Cu at (67.9, 75.8)
- added C84: 100n, Capacitor_SMD:C_0402_1005Metric, F.Cu at (67.9, 77.7)
- added C85: 100n, Capacitor_SMD:C_0402_1005Metric, F.Cu at (70.8, 54.1)
- added C86: 100n, Capacitor_SMD:C_0402_1005Metric, F.Cu at (70.8, 56.1)
- added C87: 100n, Capacitor_SMD:C_0402_1005Metric, F.Cu at (70.8, 58.0)
- added C88: 100n, Capacitor_SMD:C_0402_1005Metric, F.Cu at (70.8, 60.0)
- added C89: 100n, Capacitor_SMD:C_0402_1005Metric, F.Cu at (70.8, 62.0)
- added C9: 47u, Capacitor_SMD:C_1210_3225Metric, F.Cu at (164.6, 134.2)
- added C90: 100n, Capacitor_SMD:C_0402_1005Metric, F.Cu at (70.8, 63.9)
- added C91: NM, Capacitor_SMD:C_0402_1005Metric, F.Cu at (70.8, 65.9)
- added C92: 1p2, Capacitor_SMD:C_0402_1005Metric, F.Cu at (70.8, 67.9)
- added C93: 100n, Capacitor_SMD:C_0402_1005Metric, F.Cu at (70.8, 69.8)
- added C94: 100n, Capacitor_SMD:C_0402_1005Metric, F.Cu at (70.8, 71.8)
- added C95: 100n, Capacitor_SMD:C_0402_1005Metric, F.Cu at (70.8, 73.8)
- added C96: 1p5, Capacitor_SMD:C_0402_1005Metric, F.Cu at (70.8, 75.8)
- added C97: 2u2, Capacitor_SMD:C_0603_1608Metric, F.Cu at (62.8, 36.8)
- added C98: 100n, Capacitor_SMD:C_0402_1005Metric, F.Cu at (70.8, 77.7)
- added C99: 100n, Capacitor_SMD:C_0402_1005Metric, F.Cu at (73.7, 54.1)
- added D1: PESD5V0F1BRSF, Diode_SMD:Nexperia_DSN0603-2_0.6x0.3mm_P0.4mm, F.Cu at (93.9, 38.2)
- added D10: WS2812B, LED_SMD:LED_WS2812B_PLCC4_5.0x5.0mm_P3.2mm, F.Cu at (123.9, 67.1)
- added D11: LED, LED_SMD:LED_0603_1608Metric, F.Cu at (100.4, 71.8)
- added D12: LED, LED_SMD:LED_0603_1608Metric, F.Cu at (100.4, 74.4)
- added D13: LED, LED_SMD:LED_0603_1608Metric, F.Cu at (100.4, 77.0)
- added D14: BAV116WS, Diode_SMD:D_SOD-323, F.Cu at (124.6, 47.5)
- added D15: RClamp2451ZA, FOBtool_Custom:D_Semtech_RCLAMP2451ZA_DFN0603_2, F.Cu at (77.3, 99.5)
- added D16: PESD5V0F1BRSF, Diode_SMD:Nexperia_DSN0603-2_0.6x0.3mm_P0.4mm, F.Cu at (160.1, 62.5)
- added D17: PESD5V0F1BRSF, Diode_SMD:Nexperia_DSN0603-2_0.6x0.3mm_P0.4mm, F.Cu at (160.1, 64.1)
- added D18: PESD5V0F1BRSF, Diode_SMD:Nexperia_DSN0603-2_0.6x0.3mm_P0.4mm, F.Cu at (160.1, 65.8)
- added D19: PESD5V0F1BRSF, Diode_SMD:Nexperia_DSN0603-2_0.6x0.3mm_P0.4mm, F.Cu at (160.1, 67.4)
- added D2: RCLAMP2451ZA, FOBtool_Custom:D_Semtech_RCLAMP2451ZA_DFN0603_2, F.Cu at (77.3, 97.8)
- added D3: PESD5V0F1BRSF, Diode_SMD:Nexperia_DSN0603-2_0.6x0.3mm_P0.4mm, F.Cu at (93.9, 39.8)
- added D4: TPD1E10B06, Package_SON:Texas_DPY0002A_0.6x1mm_P0.65mm, F.Cu at (127.4, 141.7)
- added D5: TPD1E10B06, Package_SON:Texas_DPY0002A_0.6x1mm_P0.65mm, F.Cu at (127.4, 143.6)
- added D6: NUP2105L, Package_TO_SOT_SMD:SOT-23, F.Cu at (119.0, 130.1)
- added D7: LED, LED_SMD:LED_0603_1608Metric, F.Cu at (100.4, 69.2)
- added D8: WS2812B, LED_SMD:LED_WS2812B_PLCC4_5.0x5.0mm_P3.2mm, F.Cu at (123.9, 53.9)
- added D9: WS2812B, LED_SMD:LED_WS2812B_PLCC4_5.0x5.0mm_P3.2mm, F.Cu at (123.9, 60.5)
- added FB1: 600 Ω @ 100 MHz, Inductor_SMD:L_0402_1005Metric, F.Cu at (80.0, 79.7)
- added FB2: 600 Ω @ 100 MHz, Inductor_SMD:L_0402_1005Metric, F.Cu at (80.0, 81.7)
- added FB3: 600 Ω @ 100 MHz, Inductor_SMD:L_0402_1005Metric, F.Cu at (80.0, 83.7)
- added FB4: 600 Ω @ 100 MHz, Inductor_SMD:L_0402_1005Metric, F.Cu at (80.0, 85.7)
- added FB5: 600 Ω @ 100 MHz, Inductor_SMD:L_0402_1005Metric, F.Cu at (80.0, 87.7)
- added FB6: 600 Ω @ 100 MHz, Inductor_SMD:L_0402_1005Metric, F.Cu at (80.0, 89.7)
- added FB8: BLM15PX330SN1D, Inductor_SMD:L_0402_1005Metric, F.Cu at (78.4, 146.0)
- added FL10: B39871B3725U410, Filter:Filter_SAW_Epcos_DCC6C_3x3mm, F.Cu at (75.7, 81.2)
- added FL11: B39431B3710U410, Filter:Filter_SAW_Epcos_DCC6C_3x3mm, F.Cu at (75.7, 86.1)
- added FL12: B39321B3722U410, Filter:Filter_SAW_Epcos_DCC6C_3x3mm, F.Cu at (75.7, 91.0)
- added FL2: B39321B3722U410, Filter:Filter_SAW_Epcos_DCC6C_3x3mm, F.Cu at (63.9, 81.2)
- added FL3: B39431B3710U410, Filter:Filter_SAW_Epcos_DCC6C_3x3mm, F.Cu at (63.9, 86.1)
- added FL4: B39871B3725U410, Filter:Filter_SAW_Epcos_DCC6C_3x3mm, F.Cu at (63.9, 91.0)
- added FL7: B39871B3725U410, Filter:Filter_SAW_Epcos_DCC6C_3x3mm, F.Cu at (69.8, 81.2)
- added FL8: B39431B3710U410, Filter:Filter_SAW_Epcos_DCC6C_3x3mm, F.Cu at (69.8, 86.1)
- added FL9: B39321B3722U410, Filter:Filter_SAW_Epcos_DCC6C_3x3mm, F.Cu at (69.8, 91.0)
- added J1: S3B-PH-SM4-TB(LF)(SN), Connector_JST:JST_PH_S3B-PH-SM4-TB_1x03-1MP_P2.00mm_Horizontal, F.Cu at (150.4, 148.6)
- added J10: FH12-12S-0.5SH(55), Connector_FFC-FPC:Hirose_FH12-12S-0.5SH_1x12-1MP_P0.50mm_Horizontal, F.Cu at (134.6, 64.7)
- added J11: SM02B-GHS-TB(LF)(SN), Connector_JST:JST_GH_SM02B-GHS-TB_1x02-1MP_P1.25mm_Horizontal, F.Cu at (140.1, 44.9)
- added J12: Molex 104031-0811, Connector_Card:microSD_HC_Molex_104031-0811, F.Cu at (105.7, 60.8)
- added J13: U.FL-R-SMT-1(10), Connector_Coaxial:U.FL_Hirose_U.FL-R-SMT-1_Vertical, F.Cu at (70.3, 150.6)
- added J15: S2B-PH-SM4-TB(LF)(SN), Connector_JST:JST_PH_S2B-PH-SM4-TB_1x02-1MP_P2.00mm_Horizontal, F.Cu at (74.7, 108.9)
- added J16: S2B-PH-SM4-TB(LF)(SN), Connector_JST:JST_PH_S2B-PH-SM4-TB_1x02-1MP_P2.00mm_Horizontal, F.Cu at (84.9, 108.9)
- added J17: SMA5_RESERVED_CC1200, Connector_Coaxial:SMA_Amphenol_132289_EdgeMount, F.Cu at (45.8, 82.9)
- added J18: SMA6_RESERVED_DUAL_RF, Connector_Coaxial:SMA_Amphenol_132289_EdgeMount, F.Cu at (45.8, 95.2)
- added J2: M50-3530542, Connector_PinHeader_1.27mm:PinHeader_1x05_P1.27mm_Vertical, F.Cu at (166.6, 36.6)
- added J3: SMA4, Connector_Coaxial:SMA_Amphenol_132289_EdgeMount, F.Cu at (45.8, 34.1)
- added J4: SMA1_CH-A_50R, Connector_Coaxial:SMA_Amphenol_132289_EdgeMount, F.Cu at (45.8, 46.3)
- added J5: SMA2_CH-B_50R, Connector_Coaxial:SMA_Amphenol_132289_EdgeMount, F.Cu at (45.8, 58.5)
- added J6: SMA3_CH-C_50R, Connector_Coaxial:SMA_Amphenol_132289_EdgeMount, F.Cu at (45.8, 70.7)
- added J7: USB4085-GF-A_REVA4, USB4085:GCT_USB4085-GF-A_REVA4, F.Cu at (120.0, 151.6)
- added J8: USB_A, Connector_USB:USB_A_Molex_67643_Horizontal, F.Cu at (104.0, 131.2)
- added J9: SM04B-GHS-TB(LF)(SN), Connector_JST:JST_GH_SM04B-GHS-TB_1x04-1MP_P1.25mm_Horizontal, F.Cu at (119.7, 160.3)
- added L1: 2u2, Inductor_SMD:L_Wuerth_MAPI-4020, F.Cu at (141.5, 145.8)
- added L10: 11n, Inductor_SMD:L_0402_1005Metric, F.Cu at (82.9, 87.7)
- added L11: 9n1, Inductor_SMD:L_0402_1005Metric, F.Cu at (82.9, 89.7)
- added L12: 3n3, Inductor_SMD:L_0402_1005Metric, F.Cu at (82.9, 91.6)
- added L13: 6n8, Inductor_SMD:L_0402_1005Metric, F.Cu at (85.8, 79.7)
- added L14: 68n, Inductor_SMD:L_0402_1005Metric, F.Cu at (85.8, 81.7)
- added L15: 68n, Inductor_SMD:L_0402_1005Metric, F.Cu at (85.8, 83.7)
- added L16: 3n3, Inductor_SMD:L_0402_1005Metric, F.Cu at (85.8, 85.7)
- added L17: 6n8, Inductor_SMD:L_0402_1005Metric, F.Cu at (85.8, 87.7)
- added L18: 3n3, Inductor_SMD:L_0402_1005Metric, F.Cu at (85.8, 89.7)
- added L19: 6n8, Inductor_SMD:L_0402_1005Metric, F.Cu at (85.8, 91.6)
- added L2: 0u47, Inductor_SMD:L_Wuerth_MAPI-4020, F.Cu at (141.5, 151.4)
- added L20: 5n1, Inductor_SMD:L_0402_1005Metric, F.Cu at (88.7, 79.7)
- added L21: 15u, FOBtool_Custom:L_Murata_LQH44PN_4.0x4.0mm, F.Cu at (93.1, 81.6)
- added L22: 18n, Inductor_SMD:L_1008_2520Metric, F.Cu at (93.2, 64.9)
- added L23: 68n, Inductor_SMD:L_0402_1005Metric, F.Cu at (88.7, 81.7)
- added L24: 33n, Inductor_SMD:L_0603_1608Metric, F.Cu at (62.8, 51.8)
- added L25: 39n, Inductor_SMD:L_0603_1608Metric, F.Cu at (66.8, 29.3)
- added L26: 12n, Inductor_SMD:L_0603_1608Metric, F.Cu at (66.8, 31.8)
- added L27: 24n, Inductor_SMD:L_0603_1608Metric, F.Cu at (66.8, 34.3)
- added L28: 27n, Inductor_SMD:L_0603_1608Metric, F.Cu at (66.8, 36.8)
- added L29: 9n1, Inductor_SMD:L_0603_1608Metric, F.Cu at (66.8, 39.3)
- added L3: 1u, Inductor_SMD:L_Wuerth_HCI-5040, F.Cu at (152.5, 157.6)
- added L30: 12n, Inductor_SMD:L_0603_1608Metric, F.Cu at (66.8, 41.8)
- added L31: 13n, Inductor_SMD:L_0603_1608Metric, F.Cu at (66.8, 44.3)
- added L32: 3n9, Inductor_SMD:L_0603_1608Metric, F.Cu at (66.8, 46.8)
- added L33: 27n, Inductor_SMD:L_0402_1005Metric, F.Cu at (78.4, 148.0)
- added L34: 160n, Inductor_SMD:L_0603_1608Metric, F.Cu at (59.5, 109.5)
- added L35: 160n, Inductor_SMD:L_0603_1608Metric, F.Cu at (59.5, 112.0)
- added L36: 4n7, Inductor_SMD:L_0402_1005Metric, F.Cu at (88.7, 83.7)
- added L4: 3u3, FOBtool_Custom:L_Abracon_AOTA-B201610S_2.0x1.6mm, F.Cu at (165.9, 50.3)
- added L5: 20n, Inductor_SMD:L_0402_1005Metric, F.Cu at (80.0, 91.6)
- added L6: 24n, Inductor_SMD:L_0402_1005Metric, F.Cu at (82.9, 79.7)
- added L7: 15n, Inductor_SMD:L_0402_1005Metric, F.Cu at (82.9, 81.7)
- added L8: 120n, Inductor_SMD:L_0402_1005Metric, F.Cu at (82.9, 83.7)
- added L9: 11n, Inductor_SMD:L_0402_1005Metric, F.Cu at (82.9, 85.7)
- added NT1: NetTie_2, FOBtool_Custom:NetTie_2_SMD_3.0mm_Current, F.Cu at (165.8, 161.5)
- added Q1: MMBT3904, Package_TO_SOT_SMD:SOT-23, F.Cu at (119.0, 134.5)
- added Q2: MMBT3904, Package_TO_SOT_SMD:SOT-23, F.Cu at (119.0, 139.0)
- added Q3: DMN2075U-7, Package_TO_SOT_SMD:SOT-23, F.Cu at (110.0, 74.7)
- added R1: 10k, Resistor_SMD:R_0603_1608Metric, F.Cu at (144.7, 131.6)
- added R10: 32k4, Resistor_SMD:R_0603_1608Metric, F.Cu at (148.7, 139.2)
- added R100: 10k, Resistor_SMD:R_0603_1608Metric, F.Cu at (112.4, 39.3)
- added R101: 100R, Resistor_SMD:R_0603_1608Metric, F.Cu at (112.4, 41.8)
- added R102: 100R, Resistor_SMD:R_0603_1608Metric, F.Cu at (112.4, 44.3)
- added R103: 100R, Resistor_SMD:R_0603_1608Metric, F.Cu at (112.4, 46.8)
- added R104: 100k, Resistor_SMD:R_0603_1608Metric, F.Cu at (112.4, 49.3)
- added R105: 33R, Resistor_SMD:R_1206_3216Metric, F.Cu at (122.7, 76.3)
- added R106: 680R, Resistor_SMD:R_0603_1608Metric, F.Cu at (116.4, 29.3)
- added R107: 680R, Resistor_SMD:R_0603_1608Metric, F.Cu at (116.4, 31.8)
- added R108: 680R, Resistor_SMD:R_0603_1608Metric, F.Cu at (116.4, 34.3)
- added R109: 680R, Resistor_SMD:R_0603_1608Metric, F.Cu at (116.4, 36.8)
- added R11: 40k2, Resistor_SMD:R_0603_1608Metric, F.Cu at (148.7, 141.7)
- added R110: 10k, Resistor_SMD:R_0603_1608Metric, F.Cu at (116.4, 39.3)
- added R111: 10k, Resistor_SMD:R_0603_1608Metric, F.Cu at (116.4, 41.8)
- added R112: 10k, Resistor_SMD:R_0603_1608Metric, F.Cu at (116.4, 44.3)
- added R113: 10k, Resistor_SMD:R_0603_1608Metric, F.Cu at (116.4, 46.8)
- added R114: 0R, Resistor_SMD:R_0603_1608Metric, F.Cu at (59.5, 114.6)
- added R115: 0R, Resistor_SMD:R_0603_1608Metric, F.Cu at (59.5, 117.1)
- added R116: 0R, Resistor_SMD:R_0603_1608Metric, F.Cu at (59.5, 119.6)
- added R117: 0R, Resistor_SMD:R_0603_1608Metric, F.Cu at (59.5, 122.1)
- added R118: 10R, Resistor_SMD:R_0603_1608Metric, F.Cu at (59.5, 124.6)
- added R119: 10k, Resistor_SMD:R_0603_1608Metric, F.Cu at (59.5, 127.1)
- added R12: 100k, Resistor_SMD:R_0603_1608Metric, F.Cu at (152.7, 129.1)
- added R120: 100k, Resistor_SMD:R_0603_1608Metric, F.Cu at (59.5, 129.6)
- added R121: 1k, Resistor_SMD:R_0603_1608Metric, F.Cu at (63.6, 104.5)
- added R122: 1k, Resistor_SMD:R_0603_1608Metric, F.Cu at (63.6, 107.0)
- added R123: 220R, Resistor_SMD:R_0603_1608Metric, F.Cu at (63.6, 109.5)
- added R124: 4R7, Resistor_SMD:R_0805_2012Metric, F.Cu at (48.2, 132.3)
- added R125: 150k, Resistor_SMD:R_0603_1608Metric, F.Cu at (63.6, 112.0)
- added R126: 47k, Resistor_SMD:R_0603_1608Metric, F.Cu at (63.6, 114.6)
- added R127: 4R7, Resistor_SMD:R_0805_2012Metric, F.Cu at (48.2, 135.3)
- added R128: 220R, Resistor_SMD:R_0603_1608Metric, F.Cu at (63.6, 117.1)
- added R129: 4R7, Resistor_SMD:R_0805_2012Metric, F.Cu at (48.2, 138.2)
- added R13: 100k, Resistor_SMD:R_0603_1608Metric, F.Cu at (152.7, 131.6)
- added R130: 150k, Resistor_SMD:R_0603_1608Metric, F.Cu at (63.6, 119.6)
- added R131: 47k, Resistor_SMD:R_0603_1608Metric, F.Cu at (63.6, 122.1)
- added R132: 4R7, Resistor_SMD:R_0805_2012Metric, F.Cu at (48.2, 141.2)
- added R133: 2k2, Resistor_SMD:R_0603_1608Metric, F.Cu at (63.6, 124.6)
- added R134: 2k2, Resistor_SMD:R_0603_1608Metric, F.Cu at (63.6, 127.1)
- added R135: 2R7, Resistor_SMD:R_0805_2012Metric, F.Cu at (48.2, 144.1)
- added R136: 2R7, Resistor_SMD:R_0805_2012Metric, F.Cu at (48.2, 147.1)
- added R137: 6k8, Resistor_SMD:R_0603_1608Metric, F.Cu at (63.6, 129.6)
- added R138: 6k8, Resistor_SMD:R_0603_1608Metric, F.Cu at (67.6, 104.5)
- added R139: 0R, Resistor_SMD:R_0603_1608Metric, F.Cu at (82.8, 46.8)
- added R14: 43k2, Resistor_SMD:R_0603_1608Metric, F.Cu at (152.7, 134.1)
- added R140: 100k, Resistor_SMD:R_0603_1608Metric, F.Cu at (67.6, 107.0)
- added R141: 10k, Resistor_SMD:R_0603_1608Metric, F.Cu at (82.8, 49.3)
- added R142: 0R, Resistor_SMD:R_0201_0603Metric, F.Cu at (78.2, 149.9)
- added R143: 0R, Resistor_SMD:R_0201_0603Metric, F.Cu at (78.2, 151.6)
- added R144: 1k, Resistor_SMD:R_0603_1608Metric, F.Cu at (67.6, 109.5)
- added R145: 10k, Resistor_SMD:R_0603_1608Metric, F.Cu at (67.6, 112.0)
- added R146: 10k, Resistor_SMD:R_0603_1608Metric, F.Cu at (67.6, 114.6)
- added R147: 10k, Resistor_SMD:R_0603_1608Metric, F.Cu at (67.6, 117.1)
- added R148: 10k, Resistor_SMD:R_0603_1608Metric, F.Cu at (67.6, 119.6)
- added R149: 100k, Resistor_SMD:R_0603_1608Metric, F.Cu at (148.9, 63.3)
- added R15: 100k, Resistor_SMD:R_0603_1608Metric, F.Cu at (152.7, 136.7)
- added R150: 43k2, Resistor_SMD:R_0603_1608Metric, F.Cu at (148.9, 65.9)
- added R151: 100k, Resistor_SMD:R_0603_1608Metric, F.Cu at (152.9, 55.8)
- added R152: 33R, Resistor_SMD:R_0603_1608Metric, F.Cu at (152.9, 58.3)
- added R153: 100k, Resistor_SMD:R_0603_1608Metric, F.Cu at (152.9, 60.8)
- added R154: 33R, Resistor_SMD:R_0603_1608Metric, F.Cu at (152.9, 63.3)
- added R155: 100k, Resistor_SMD:R_0603_1608Metric, F.Cu at (152.9, 65.9)
- added R156: 33R, Resistor_SMD:R_0603_1608Metric, F.Cu at (156.9, 55.8)
- added R157: 10k, Resistor_SMD:R_0603_1608Metric, F.Cu at (156.9, 58.3)
- added R158: 1k, Resistor_SMD:R_0603_1608Metric, F.Cu at (156.9, 60.8)
- added R16: 732k, Resistor_SMD:R_0603_1608Metric, F.Cu at (152.7, 139.2)
- added R17: 100k, Resistor_SMD:R_0603_1608Metric, F.Cu at (152.7, 141.7)
- added R18: 10k, Resistor_SMD:R_0603_1608Metric, F.Cu at (149.4, 86.5)
- added R19: 10k, Resistor_SMD:R_0603_1608Metric, F.Cu at (149.4, 89.1)
- added R2: 261R, Resistor_SMD:R_0603_1608Metric, F.Cu at (144.7, 134.1)
- added R20: 2k2, Resistor_SMD:R_0603_1608Metric, F.Cu at (149.4, 91.6)
- added R21: 2k2, Resistor_SMD:R_0603_1608Metric, F.Cu at (149.4, 94.1)
- added R22: 499R, Resistor_SMD:R_0603_1608Metric, F.Cu at (149.4, 96.6)
- added R23: 10k, Resistor_SMD:R_0603_1608Metric, F.Cu at (149.4, 99.1)
- added R24: 33R, Resistor_SMD:R_0603_1608Metric, F.Cu at (148.9, 36.8)
- added R25: 1k, Resistor_SMD:R_0603_1608Metric, F.Cu at (148.9, 39.3)
- added R26: 27R, Resistor_SMD:R_0603_1608Metric, F.Cu at (148.9, 41.8)
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Other:
- board outline added: 64 x 112 mm

Commit message: all 3d models finished except t1-t3 and start initial placement
Parts:
- moved SW1 181.7 mm to (285.0, 127.0)
Other:
- board text added: "DISPLAY BODY 34.60 x 47.80 mm PROVISIONAL POSITION"
Changed lines of the file:
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@@
 		)
 		(embedded_fonts no)
+		(model "${KIPRJMOD}/Custom_Components/CS/CSTCR4M00G55B-R0/CSTCR4M00G55B-R0.step"
+			(offset
+				(xyz 0 0 0)
+			)
+			(scale
+				(xyz 1 1 1)
+			)
+			(rotate
+				(xyz -90 -0 -0)
+			)
+		)
 	)
 	(footprint "Capacitor_SMD:C_0402_1005Metric"
@@
 		)
 		(embedded_fonts no)
+		(model "${KIPRJMOD}/Custom_Components/FOBtool_Custom/3dmodels/EEFLR0J680R.step"
+			(offset
+				(xyz 0.05 0 0)
+			)
+			(scale
+				(xyz 1 1 1)
+			)
+			(rotate
+				(xyz -90 -0 -0)
+			)
+		)
 	)
 	(footprint "Filter:Filter_SAW_Epcos_DCC6C_3x3mm"
@@
 		)
 		(embedded_fonts no)
+		(model "${KIPRJMOD}/Custom_Components/SN/SN74AHCT00PWR/SN74AHCT00PWR.step"
+			(offset
+				(xyz 0 0 0)
+			)
+			(scale
+				(xyz 1 1 1)
+			)
+			(rotate
+				(xyz -90 -0 -0)
+			)
+		)
 	)
 	(footprint "Crystal:Crystal_SMD_3225-4Pin_3.2x2.5mm"
@@
 		)
 		(embedded_fonts no)
+		(model "${KIPRJMOD}/Custom_Components/FOBtool_Custom/3dmodels/SLP0603P2X3F_SEM.step"
+			(offset
+				(xyz 0 0 0)
+			)
+			(scale
+				(xyz 1 1 1)
+			)
+			(rotate
+				(xyz 0 0 0)
+			)
+		)
 	)
 	(footprint "Resistor_SMD:R_0603_1608Metric"
@@
 		)
 		(embedded_fonts no)
+		(model "${KIPRJMOD}/Custom_Components/FOBtool_Custom/3dmodels/BGS13SN8E6327XTSA1.stp"
+			(offset
+				(xyz 0 0 0.02)
+			)
+			(scale
+				(xyz 1 1 1)
+			)
+			(rotate
+				(xyz -90 -0 -180)
+			)
+		)
 	)
 	(footprint "Resistor_SMD:R_0603_1608Metric"
@@
 		)
 		(embedded_fonts no)
+		(model "${KIPRJMOD}/Custom_Components/FOBtool_Custom/3dmodels/BGS13SN8E6327XTSA1.stp"
+			(offset
+				(xyz 0 0 0.02)
+			)
+			(scale
+				(xyz 1 1 1)
+			)
+			(rotate
+				(xyz -90 -0 -180)
+			)
+		)
 	)
 	(footprint "Resistor_SMD:R_0201_0603Metric"
@@
 		)
 		(embedded_fonts no)
+		(model "${KIPRJMOD}/Custom_Components/CS/CSTCR4M00G55B-R0/CSTCR4M00G55B-R0.step"
+			(offset
+				(xyz 0 0 0)
+			)
+			(scale
+				(xyz 1 1 1)
+			)
+			(rotate
+				(xyz -90 -0 -0)
+			)
+		)
 	)
 	(footprint "Inductor_SMD:L_0402_1005Metric"
@@
 		)
 		(embedded_fonts no)
+		(model "${KIPRJMOD}/Custom_Components/FOBtool_Custom/3dmodels/BGS13SN8E6327XTSA1.stp"
+			(offset
+				(xyz 0 0 0.02)
+			)
+			(scale
+				(xyz 1 1 1)
+			)
+			(rotate
+				(xyz -90 -0 -180)
+			)
+		)
 	)
 	(footprint "Capacitor_SMD:C_0402_1005Metric"
@@
 		)
 		(embedded_fonts no)
+		(model "${KIPRJMOD}/Custom_Components/FOBtool_Custom/3dmodels/BGS13SN8E6327XTSA1.stp"
+			(offset
+				(xyz 0 0 0.02)
+			)
+			(scale
+				(xyz 1 1 1)
+			)
+			(rotate
+				(xyz -90 -0 -180)
+			)
+		)
 	)
 	(footprint "Crystal:Crystal_SMD_3215-2Pin_3.2x1.5mm"
@@
 		)
 		(embedded_fonts no)
+		(model "${KIPRJMOD}/Custom_Components/LT/LT3154AV_TRPBF/LT3154AV_TRPBF.step"
+			(offset
+				(xyz 0 0 0)
+			)
+			(scale
+				(xyz 1 1 1)
+			)
+			(rotate
+				(xyz -90 -0 -0)
+			)
+		)
 	)
 	(footprint "Resistor_SMD:R_0603_1608Metric"
@@
 		)
 		(embedded_fonts no)
+		(model "${KIPRJMOD}/Custom_Components/FOBtool_Custom/3dmodels/SLP0603P2X3F_SEM.step"
+			(offset
+				(xyz 0 0 0)
+			)
+			(scale
+				(xyz 1 1 1)
+			)
+			(rotate
+				(xyz 0 0 0)
+			)
+		)
 	)
 	(footprint "Inductor_SMD:L_0402_1005Metric"
@@
 	(footprint "FOBtool_Custom:RotaryEncoder_Bourns_PEC11R-4215F-S0024"
 		(layer "F.Cu")
-		(at 127.245 36.775)
+		(at 285 127)
 		(descr "Bourns PEC11R-4215F-S0024 12 mm incremental rotary encoder, rear-facing through-hole terminals, 15 mm flatted shaft, 24 detents, 24 pulses and momentary push switch")
 		(tags "Bourns PEC11R PEC11R-4215F-S0024 rotary encoder push switch rear facing through hole")
@@
 		)
 		(embedded_fonts no)
+		(model "${KIPRJMOD}/Custom_Components/TQP/TQP3M9036/TQP3M9036.step"
+			(offset
+				(xyz 0 0 0)
+			)
+			(scale
+				(xyz 1 1 1)
+			)
+			(rotate
+				(xyz -90 -0 -0)
+			)
+		)
 	)
 	(footprint "Inductor_SMD:L_0402_1005Metric"
@@
 		)
 		(embedded_fonts no)
+		(model "${KIPRJMOD}/Custom_Components/FOBtool_Custom/3dmodels/CPH3225A.step"
+			(offset
+				(xyz 0 0 0)
+			)
+			(scale
+				(xyz 1 1 1)
+			)
+			(rotate
+				(xyz -90 -0 -0)
+			)
+		)
 	)
 	(footprint "Capacitor_SMD:C_0402_1005Metric"
@@
 		)
 		(embedded_fonts no)
+		(model "${KIPRJMOD}/Custom_Components/FOBtool_Custom/3dmodels/LQH44PN150MPRL.step"
+			(offset
+				(xyz 0 0 0)
+			)
+			(scale
+				(xyz 1 1 1)
+			)
+			(rotate
+				(xyz -90 -0 -0)
+			)
+		)
 	)
 	(footprint "LED_SMD:LED_0603_1608Metric"
@@
 		)
 		(embedded_fonts no)
+		(model "${KIPRJMOD}/Custom_Components/FOBtool_Custom/3dmodels/BGS13SN8E6327XTSA1.stp"
+			(offset
+				(xyz 0 0 0.02)
+			)
+			(scale
+				(xyz 1 1 1)
+			)
+			(rotate
+				(xyz -90 -0 -180)
+			)
+		)
 	)
 	(footprint "Capacitor_SMD:C_0805_2012Metric"
@@
 		)
 		(embedded_fonts no)
+		(model "${KIPRJMOD}/Custom_Components/FOBtool_Custom/3dmodels/BGS13SN8E6327XTSA1.stp"
+			(offset
+				(xyz 0 0 0.02)
+			)
+			(scale
+				(xyz 1 1 1)
+			)
+			(rotate
+				(xyz -90 -0 -180)
+			)
+		)
 	)
 	(footprint "Capacitor_SMD:C_0402_1005Metric"
@@
 		)
 		(embedded_fonts no)
+		(model "${KIPRJMOD}/Custom_Components/FOBtool_Custom/3dmodels/AOTA-B201610S3R3-101-T--3DModel-STEP-510211.STEP"
+			(offset
+				(xyz 0 0 0)
+			)
+			(scale
+				(xyz 1 1 1)
+			)
+			(rotate
+				(xyz -90 -0 -0)
+			)
+		)
 	)
 	(footprint "Resistor_SMD:R_0603_1608Metric"
@@
 		)
 		(embedded_fonts no)
+		(model "${KIPRJMOD}/Custom_Components/FOBtool_Custom/3dmodels/EEFTX0J121RF.step"
+			(offset
+				(xyz 0 0 0)
+			)
+			(scale
+				(xyz 1 1 1)
+			)
+			(rotate
+				(xyz -90 -0 -0)
+			)
+		)
 	)
 	(footprint "Capacitor_SMD:C_0603_1608Metric"
@@
 		(layer "Dwgs.User")
 	)
+	(gr_rect
+		(start 267.7 65)
+		(end 302.3 112.8)
+		(stroke
+			(width 0.1)
+			(type solid)
+		)
+		(fill no)
+		(layer "Dwgs.User")
+	)
 	(gr_line
 		(start 285 53)
@@
 		(layer "Edge.Cuts")
 	)
+	(gr_text "DISPLAY BODY 34.60 x 47.80 mm\nPROVISIONAL POSITION"
+		(at 274 69 0)
+		(layer "Dwgs.User")
+		(effects
+			(font
+				(size 1 1)
+				(thickness 0.15)
+			)
+			(justify left bottom)
+		)
+	)
 	(embedded_fonts no)

Commit message: grouped the sheets together for placement
Parts:
- moved J4 392.8 mm to (433.7, 108.0)
- moved D13 391.2 mm to (487.0, 17.0)
- moved J5 387.5 mm to (426.1, 132.9)
- moved D12 379.9 mm to (476.0, 17.0)
- moved SW8 376.4 mm to (488.3, 13.4)
- moved R109 375.1 mm to (491.0, 17.0)
- moved C73 370.9 mm to (429.0, 143.1)
- moved C74 370.9 mm to (429.0, 145.0)
- moved C75 370.9 mm to (429.0, 147.0)
- moved C71 369.6 mm to (426.1, 145.0)
- moved C72 369.6 mm to (426.1, 147.0)
- moved D11 368.7 mm to (465.0, 17.0)
- moved L25 367.3 mm to (419.8, 130.6)
- moved L26 367.3 mm to (419.8, 133.1)
- moved L27 367.3 mm to (419.8, 135.6)
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
Commit message: adding provisional space
Parts:
- moved J18 267.8 mm to (305.0, 162.5), turned to -90 degrees
- moved J17 260.7 mm to (305.0, 55.5), turned to 90 degrees
- moved SW3 228.9 mm to (267.0, 145.0)
- moved SW4 228.9 mm to (279.0, 145.0)
- moved SW5 228.1 mm to (291.0, 145.0)
- moved SW8 227.3 mm to (303.0, 145.0)
- moved J9 199.0 mm to (313.5, 137.0), turned to 90 degrees
- moved J4 176.7 mm to (265.0, 55.5), turned to 90 degrees
- moved J5 163.8 mm to (265.0, 162.5), turned to -90 degrees
- moved J6 155.1 mm to (285.0, 55.5), turned to 90 degrees
- moved D10 154.1 mm to (293.0, 62.0)
- moved D9 151.1 mm to (285.0, 62.0)
- moved D8 144.9 mm to (277.0, 62.0)
- moved J8 134.9 mm to (307.7, 103.5), turned to 90 degrees
- moved J7 132.3 mm to (315.3, 80.0), turned to 90 degrees
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Other:
- board text added: "BATTERY MAX BODY"
- board text added: "DISPLAY FPC / J10. PROVISIONAL SERVICE AREA."
- board text added: "M2 MOUNT Ø6"
- board text added: "NANO-FIT MATED ENVELOPE"
- board text added: "REAR BATTERY UNPLUG ACCESS"
- board text added: "REAR DOCK BAY 40 × 30 mm"
- board text added: "REAR NFC + LF COILS SHARED AREA"
