File: FOBtool_HW.kicad_pcb (KiCad board)
At the start: 6 copper layers, 64 x 112 mm, 591 parts, among them J1 S3B-PH-SM4-TB(LF)(SN), J10 FH12-12S-0.5SH(55), J11 SM02B-GHS-TB(LF)(SN), J12 Molex 104031-0811, J13 U.FL-R-SMT-1(10), J15 S2B-PH-SM4-TB(LF)(SN), J16 S2B-PH-SM4-TB(LF)(SN), J17 SMA5_RESERVED_CC1200, J18 SMA6_RESERVED_DUAL_RF, J2 M50-3530542, J3 SMA4, J4 SMA1_CH-A_50R, J5 SMA2_CH-B_50R, J6 SMA3_CH-C_50R, J7 USB4085-GF-A_REVA4, J8 USB_A, J9 SM04B-GHS-TB(LF)(SN), Q1 MMBT3904, Q2 MMBT3904, Q3 DMN2075U-7, SW1 RotaryEncoder_Switch, SW2 SW_Push, SW3 SW_Push, SW4 SW_Push, SW5 SW_Push, SW6 SW_Push, SW7 SW_Push, SW8 SW_Push, T1 B0310J50100AHF, T2 B0310J50100AHF, T3 B0310J50100AHF, U1 ESP32-S3-WROOM-1-N16R2, U10 BGS12WN6E6327XTSA1, U11 MAX17048G+, U12 BGS12WN6E6327XTSA1, U13 BQ25895RTW, U14 TQP3M9036, U15 TSS-13LN+, U16 TCA9535PWR, U17 TQP3M9036, U18 BGS13SN8E6327XTSA1, U19 BGS13SN8E6327XTSA1, U2 RP2350A, U20 BGS13SN8E6327XTSA1, U21 BGS13SN8E6327XTSA1, U22 TQP7M9106, U23 LT3154AV#TRPBF, U25 TPS2553DBVR, U26 W25Q128JVSIQ, U27 TPS22918DBVR, U28 BGS12P2L6, U29 BGS12P2L6, U3 CC1101RGPR, U30 BGS12P2L6, U31 BGS12P2L6, U32 TPD2E2U06DCK, U33 CP2102N-Axx-xQFN24, U34 TPD2E2U06DCK, U35 DW3220, U36 SN65HVD230, U37 SN74AHCT1G125DBVR, U38 DRV2605LDGS, U39 TCA9534PWR, U4 CC1101RGPR, U40 ATECC608C-TCSM, U41 MAX-M10N-10B-00, U42 LTR-303ALS-01, U43 PCF85263AT/AJ, U44 PN7160B1HN/C100E, U45 TMS3705FDRQ1, U46 TMS3705FDRQ1, U47 SN74AHCT00PWR, U48 SN74LVC157APWR, U49 TPS61022, U5 CC1101RGPR, U50 TPS2553DBVR, U6 SI4463-C2A-GM, U7 BGS12WN6E6327XTSA1, U8 BGS13SN8E6327XTSA1, U9 BGS13SN8E6327XTSA1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

Commit message: finished initial placement for rp2350A and esp32
Parts:
- added J_BAT_FIT: 105430-1203, 1054:CONN_SD-105430-001_03_MOL, B.Cu at (309.0, 115.0)
- C2, C6: moved to B.Cu
- moved C7 306.1 mm to (293.9, 293.9), turned to 180 degrees
- moved C2 169.0 mm to (294.7, 134.1)
- moved C1 164.2 mm to (293.2, 136.2)
- moved C5 164.1 mm to (301.5, 138.5), turned to -90 degrees
- moved C4 159.9 mm to (301.5, 130.5), turned to -90 degrees
- moved C3 157.9 mm to (298.0, 133.6)
- moved C6 157.6 mm to (302.0, 138.5), turned to 90 degrees
- moved L1 152.9 mm to (297.0, 130.2), turned to 90 degrees
- moved U13 151.0 mm to (297.5, 137.5)
- moved U33 150.7 mm to (303.0, 80.0), turned to 180 degrees
- moved C153 145.2 mm to (308.2, 77.0), turned to 90 degrees
- moved C154 143.6 mm to (306.5, 77.0), turned to 90 degrees
- moved C150 142.6 mm to (309.0, 85.5), turned to -90 degrees
- moved C155 141.9 mm to (302.2, 75.7), turned to 90 degrees
- moved C156 138.9 mm to (303.9, 75.7), turned to 90 degrees
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Other:
- board text added: "BATTERY CONNECTOR OPENING"

Commit message: finished the rf control group initial placement
Parts:
- added C133: 100n, Capacitor_SMD:C_0402_1005Metric, F.Cu at (295.0, 93.0)
- C157, NT1: moved to B.Cu
- C2, C6: moved to F.Cu
- moved C12 207.4 mm to (266.4, 141.2), turned to 180 degrees
- moved C11 206.8 mm to (271.5, 141.2), turned to 180 degrees
- moved C160 201.5 mm to (313.0, 137.5), turned to 90 degrees
- moved L2 199.9 mm to (267.9, 137.0), turned to 90 degrees
- moved D6 198.2 mm to (308.0, 145.0)
- moved C13 197.3 mm to (276.5, 140.5), turned to -90 degrees
- moved C8 196.2 mm to (271.5, 132.6), turned to 180 degrees
- moved C9 196.2 mm to (266.4, 132.6), turned to 180 degrees
- moved R84 194.4 mm to (316.0, 131.5), turned to -90 degrees
- moved R85 193.7 mm to (313.0, 134.3), turned to -90 degrees
- moved C14 190.9 mm to (277.1, 135.5), turned to 180 degrees
- moved C159 190.5 mm to (311.5, 124.0), turned to 180 degrees
- moved C10 190.2 mm to (266.4, 128.8), turned to 180 degrees
- moved R86 189.6 mm to (310.0, 133.5)
- moved U23 188.7 mm to (273.0, 137.0), turned to 90 degrees
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