File: FOBtool_HW.kicad_pcb (KiCad board)
At the start: 6 copper layers, 64 x 112 mm, 595 parts, among them J1 S3B-PH-SM4-TB(LF)(SN), J10 FH12-12S-0.5SH(55), J11 SM02B-GHS-TB(LF)(SN), J12 Molex 104031-0811, J13 U.FL-R-SMT-1(10), J15 S2B-PH-SM4-TB(LF)(SN), J16 S2B-PH-SM4-TB(LF)(SN), J17 SMA5_RESERVED_CC1200, J18 SMA6_RESERVED_DUAL_RF, J2 M50-3530542, J21 781710002, J22 78171-5006, J3 SMA4, J4 SMA1_CH-A_50R, J5 SMA2_CH-B_50R, J6 SMA3_CH-C_50R, J7 USB4085-GF-A_REVA4, J8 USB_A, J9 SM04B-GHS-TB(LF)(SN), Q1 MMBT3904, Q2 MMBT3904, Q3 DMN2075U-7, SW1 RotaryEncoder_Switch, SW2 SW_Push, SW3 SW_Push, SW4 SW_Push, SW5 SW_Push, SW6 SW_Push, SW7 SW_Push, SW8 SW_Push, T1 B0310J50100AHF, T2 B0310J50100AHF, T3 B0310J50100AHF, U1 ESP32-S3-WROOM-1-N16R2, U10 BGS12WN6E6327XTSA1, U11 MAX17048G+, U12 BGS12WN6E6327XTSA1, U13 BQ25895RTW, U14 TQP3M9036, U15 TSS-13LN+, U16 TCA9535PWR, U17 TQP3M9036, U18 BGS13SN8E6327XTSA1, U19 BGS13SN8E6327XTSA1, U2 RP2350A, U20 BGS13SN8E6327XTSA1, U21 BGS13SN8E6327XTSA1, U22 TQP7M9106, U23 LT3154AV#TRPBF, U25 TPS2553DBVR, U26 W25Q128JVSIQ, U27 TPS22918DBVR, U28 BGS12P2L6, U29 BGS12P2L6, U3 CC1101RGPR, U30 BGS12P2L6, U31 BGS12P2L6, U32 TPD2E2U06DCK, U33 CP2102N-Axx-xQFN24, U34 TPD2E2U06DCK, U35 DW3220, U36 SN65HVD230, U37 SN74AHCT1G125DBVR, U38 DRV2605LDGS, U39 TCA9534PWR, U4 CC1101RGPR, U40 ATECC608C-TCSM, U41 MAX-M10N-10B-00, U42 LTR-303ALS-01, U43 PCF85263AT/AJ, U44 PN7160B1HN/C100E, U45 TMS3705FDRQ1, U46 TMS3705FDRQ1, U47 SN74AHCT00PWR, U48 SN74LVC157APWR, U49 TPS61022, U5 CC1101RGPR, U50 TPS2553DBVR, U6 SI4463-C2A-GM, U7 BGS12WN6E6327XTSA1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

Commit message: first revision before changing spi
Parts:
- added H1: MountingHole, MountingHole:MountingHole_2.2mm_M2, F.Cu at (256.0, 57.0)
- added H2: MountingHole, MountingHole:MountingHole_2.2mm_M2, F.Cu at (314.0, 57.0)
- added H3: MountingHole, MountingHole:MountingHole_2.2mm_M2, F.Cu at (256.0, 161.0)
- added H4: MountingHole, MountingHole:MountingHole_2.2mm_M2, F.Cu at (314.0, 161.0)
- moved C161 117.4 mm to (313.1, 17.6)
- moved C162 117.4 mm to (314.1, 23.6)
- moved C163 117.4 mm to (312.1, 23.6)
- moved J10 117.4 mm to (318.6, 19.6)
Other:
- board text added: "Candidate swollen pack: 49.5 × 94 × 5.3 mm - tolerances and lead exit pending"
- board text removed: "BATTERY CONNECTOR OPENING"
- board text removed: "NANO-FIT MATED ENVELOPE"
- board text removed: "REAR BATTERY UNPLUG ACCESS"
