File: ANCHOR_DOCK.kicad_sch (KiCad schematic)
At the start: 22 parts, among them J14 J-DOCK_8P_CUSTOM_POGO, U50 TPS2553DBVR

Commit message: the schematic is finished
Parts:
- J14: DISTRIBUTOR_LINK (none) -> N/A; MANUFACTURER (none) -> N/A; MPN (none) -> N/A
Connections:
- net DOCK_VBUS: now also J14.8 (Pin_8)
- net GND: now also J14.7 (Pin_7)
- no-connect marks 2 -> 0
Changed lines of the file:
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@@
 	)
 	(rectangle
-		(start 12.7 15.24)
-		(end 162.56 74.93)
+		(start 12.7 12.7)
+		(end 162.56 77.47)
 		(stroke
 			(width 0)
@@
 	(text "J-DOCK CONTACT SEQUENCE: \n	pins 1/2/7/8 are long power/ground contacts; pins 3/4/5 are medium signal contacts; \n	pin 6 DOCK_SENSE is the shortest contact. DOCK_VBUS remains disabled until DOCK_SENSE is debounced LOW. \n	On removal, disable DOCK_VBUS when DOCK_SENSE becomes HIGH. \n	Dock UART operates at 921600 baud using the existing framed CRC protocol."
 		(exclude_from_sim no)
-		(at 168.402 108.712 0)
+		(at 170.18 94.742 0)
 		(effects
 			(font
@@
 	)
 	(junction
+		(at 107.95 127)
+		(diameter 0)
+		(color 0 0 0 0)
+	)
+	(junction
 		(at 72.39 163.83)
 		(diameter 0)
@@
 		(color 0 0 0 0)
 	)
-	(no_connect
-		(at 130.81 127)
-	)
-	(no_connect
-		(at 130.81 129.54)
-	)
 	(wire
 		(pts
@@
 	(wire
 		(pts
+			(xy 107.95 127) (xy 130.81 127)
+		)
+		(stroke
+			(width 0)
+			(type default)
+		)
+	)
+	(wire
+		(pts
 			(xy 71.12 96.52) (xy 71.12 100.33)
 		)
@@
 	(wire
 		(pts
+			(xy 119.38 129.54) (xy 130.81 129.54)
+		)
+		(stroke
+			(width 0)
+			(type default)
+		)
+	)
+	(wire
+		(pts
 			(xy 121.92 96.52) (xy 121.92 99.06)
 		)
@@
 	(wire
 		(pts
+			(xy 107.95 127) (xy 107.95 132.08)
+		)
+		(stroke
+			(width 0)
+			(type default)
+		)
+	)
+	(wire
+		(pts
 			(xy 46.99 130.81) (xy 46.99 128.27)
 		)
@@
 	(wire
 		(pts
-			(xy 107.95 114.3) (xy 107.95 132.08)
+			(xy 107.95 114.3) (xy 107.95 127)
 		)
 		(stroke
@@
 	)
 	(label "DOCK_VBUS"
+		(at 119.38 129.54 0)
+		(effects
+			(font
+				(size 1.27 1.27)
+			)
+			(justify left bottom)
+		)
+	)
+	(label "DOCK_VBUS"
 		(at 93.98 45.72 0)
 		(effects
@@
 			)
 		)
-		(property "Datasheet" ""
+		(property "Datasheet" "N/A"
 			(at 135.89 119.38 0)
 			(hide yes)
@@
 			(at 135.89 119.38 0)
 			(hide yes)
+			(show_name no)
+			(do_not_autoplace no)
+			(effects
+				(font
+					(size 1.27 1.27)
+				)
+			)
+		)
+		(property "DISTRIBUTOR_LINK" "N/A"
+			(at 135.89 119.38 0)
+			(hide yes)
+			(show_name no)
+			(do_not_autoplace no)
+			(effects
+				(font
+					(size 1.27 1.27)
+				)
+			)
+		)
+		(property "MANUFACTURER" "N/A"
+			(at 135.89 119.38 0)
+			(hide yes)
+			(show_name no)
+			(do_not_autoplace no)
+			(effects
+				(font
+					(size 1.27 1.27)
+				)
+			)
+		)
+		(property "MPN" "N/A"
+			(at 135.89 119.38 0)
+			(hide yes)

Commit message: finished schematic phase
Changed lines of the file:
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@@
 	(text "J-DOCK CONTACT SEQUENCE: \n	pins 1/2/7/8 are long power/ground contacts; pins 3/4/5 are medium signal contacts; \n	pin 6 DOCK_SENSE is the shortest contact. DOCK_VBUS remains disabled until DOCK_SENSE is debounced LOW. \n	On removal, disable DOCK_VBUS when DOCK_SENSE becomes HIGH. \n	Dock UART operates at 921600 baud using the existing framed CRC protocol."
 		(exclude_from_sim no)
-		(at 170.18 94.742 0)
+		(at 167.64 21.082 0)
 		(effects
 			(font

Commit message: nearly finishing placement phase
Parts:
- added J22: 78171-5006, FOBtool_Connectors:Molex_78171-5006_1x06_P1.20mm, symbol Connector_Generic:Conn_01x06
Connections:
- net DOCK_LINK_A_RAW: now also J22.3 (Pin_3)
- net DOCK_LINK_B_RAW: now also J22.4 (Pin_4)
- net DOCK_SENSE_RAW: now also J22.6 (Pin_6)
- net DOCK_SYNC_RAW: now also J22.5 (Pin_5)
- net DOCK_VBUS: now also J22.1 (Pin_1)
- net GND: now also J22.2 (Pin_2)
