File: POSITIONING.kicad_sch (KiCad schematic)
At the start: 121 parts, among them J13 Conn_Coaxial, U35 DW3220, U41 MAX-M10N-10B, U44 PN7160B1HN/C101Y, U45 TMS3705FDRQ1, U46 TMS3705FDRQ1, U47 SN74AHCT00PWR, U48 SN74LVC157APWR, Y10 CSTCR4M00G55B-R0, Y7 TXC 8Y38472012, Y8 NX2016SA-27.12MHZ-EXS00A-CS06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, Y9 CSTCR4M00G55B-R0

Commit message: finished annotation
Parts:
- U41: value MAX-M10N-10B -> MAX-M10N-10B-00
- U47: footprint SN74AHCT00PWR:SOP65P640X120-14N -> SN74:SOP65P640X120-14N
- U48: footprint SN74LVC157APWR:SOP65P640X120-16N -> Package_SO:TSSOP-16_4.4x5mm_P0.65mm
- Y10, Y9: footprint CSTCR4M00G55B-R0:OSC_CSTCR4M00G55B-R0 -> CSCT:OSC_CSTCR4M00G55B-R0
- Y8: value NX2016SA-27.12MHZ-EXS00A-CS06346 -> NX2016SA 27.12MHz EXS00A-CS06346
- renumbered C186 to C183, C183 to C184, C184 to C185, C185 to C186, C182 to C187, C163 to C188, C162 to C189, C189 to C190, C188 to C191, C187 to C192, C190 to C193, C191 to C194, C192 to C195, C193 to C196, C198 to C197, C199 to C198, C196 to C199, C197 to C200, C195 to C201, C194 to C202, C200 to C203, C201 to C204, C202 to C205, C251 to C206, C250 to C207, C253 to C208, C240 to C209, C241 to C210, C243 to C211, C244 to C212, C254 to C213, C255 to C214, C256 to C215, C242 to C216, C245 to C217, C247 to C218, C230 to C219, C231 to C220, C232 to C221, C233 to C222, C237 to C223, C238 to C224, C239 to C225, C252 to C226, C234 to C227, C235 to C228, C236 to C229, C208 to C230, C207 to C231, C211 to C232, C209 to C233, C210 to C234, C228 to C235, C229 to C236, C203 to C237, C204 to C238, C214 to C239, C215 to C240, C216 to C241, C217 to C242, C218 to C243, C219 to C244, C220 to C245, C221 to C246, C222 to C247, C223 to C248, C224 to C249, C225 to C250, C227 to C251, C226 to C252, C212 to C253, C213 to C254, C205 to C255, C206 to C256, R117 to R114, R90 to R115, R89 to R116, R87 to R117, R133 to R119, R134 to R120, R135 to R121, R136 to R122, R137 to R123, R129 to R124, R130 to R125, R131 to R126, R132 to R127, R138 to R128, R125 to R129, R128 to R130, R127 to R131, R126 to R132, R121 to R133, R122 to R134, R119 to R135, R120 to R136, R123 to R137, R124 to R138
Connections:
- net NFC_VBAT is gone; now on net +5V_SYS: U44.12 (VBAT2)
- net UWB_RF2_IC: now reaches C199.1, U35.13 (RF2)
- net UWB_RF2_MATCH: now reaches C199.2, R115.1
- net UWB_ANT2_PORT: now reaches AE1.1 (A), C200.1, R115.2
- net TMS_B_ANT1: now reaches R124.1, U46.5 (ANT1)
- net UWB_XTI_IC: now reaches R116.1, U35.21 (XTI)
- net UWB_XTI_XTAL: now reaches C201.1, R116.2, Y7.3
- net UWB_ANT1_PORT: now reaches AE2.1 (A), C198.1, R114.2
- net UWB_XTO_IC: now reaches R117.1, U35.22 (XTO)
- net UWB_XTO_XTAL: now reaches C202.1, R117.2, Y7.1
- net NFC_ANT_LOOP_P: now reaches AE3.1, R135.2
- net UWB_RF1_IC: now reaches C197.1, U35.18 (RF1)
- net UWB_RF1_MATCH: now reaches C197.2, R114.1
- net GNSS_ANT_BIAS_FILT: now reaches C205.2, L33.1, R118.2
- net TMS_A_ANT1: now reaches R129.1, U45.5 (ANT1)
- net NFC_ANT_LOOP_N: now reaches AE3.2, R136.2
- net GNSS_VCC_RF: now reaches R118.1, U41.14 (VCC_RF)
- net UWB_VIO_D: now reaches C196.1, U35.38 (VIO_D)
- net MAX_RF_IN renamed GNSS_RF_IN
- net NFC_ANT_N renamed NFC_MATCH_OUT_N
- net NFC_ANT_P renamed NFC_MATCH_OUT_P
- net RX_N_NODE renamed NFC_RX_MATCH_N
- net RX_P_NODE renamed NFC_RX_MATCH_P
- net SN_1A renamed LF_SCIO_A_MUX_IN
- net SN_1B renamed LF_SCIO_B_MUX_IN
- net TX1_EMC renamed NFC_TX1_EMC
- net TX2_EMC renamed NFC_TX2_EMC
- net VTX_D renamed UWB_VTX_D
Other:
- note added: "GNSS RECEIVER, ACTIVE-ANTENNA BIAS AND SMA"
- note added: "LF COIL SELECT, TXCT GATING AND SCIO MUX"
- note added: "LF HDX 134.2 kHz — COIL A"
- note added: "LF HDX 134.2 kHz — COIL B"
- note added: "NFC CONTROLLER, MATCHING, FIELD DETECTOR AND LOOP ANTENNA"
- note added: "UWB TRANSCEIVER, CLOCK, DUAL ANTENNAS AND SPI"
- note removed: "UWB transceiver: supplies, ground and reference clock"
- title: (none) -> UWB, GNSS, NFC and LF Positioning / Credential Interfaces
- moved on the sheet: AE3, C199, FB8, L33, R118, R124, R129, R134

Commit message: finished ANCHOR_DOCK sheet
Parts:
- removed AE1, AE2: Antenna, symbol Device:Antenna
- removed FB7: BLM15AG601SN1D, symbol Device:FerriteBead
- added AE1, AE2: UWA.01, symbol FOBtool_Custom:UWA.01
- added AE4: ADFGP.25E.07.0060A, symbol Device:Antenna
- added C257, C258: DNP, Capacitor_SMD:C_0402_1005Metric, symbol Device:C
- added J15, J16: S2B-PH-SM4-TB(LF)(SN), Connector_JST:JST_PH_S2B-PH-SM4-TB_1x02-1MP_P2.00mm_Horizontal, symbol Connector_Generic:Conn_01x02
- added J19, J20: PHR-2, symbol Connector_Generic:Conn_01x02
- added MP1, MP2, MP3, MP4: SPH-002T-P0.5S, symbol Connector_Generic:Conn_01x01
- added R140: 100k, Resistor_SMD:R_0603_1608Metric, symbol Device:R
- added R142, R143: 0R, Resistor_SMD:R_0201_0603Metric, symbol Device:R
- added R144: 1k, Resistor_SMD:R_0603_1608Metric, symbol Device:R
- added R145, R146, R147, R148: 10k, Resistor_SMD:R_0603_1608Metric, symbol Device:R
- AE3: DISTRIBUTOR_LINK (none) -> N/A; MANUFACTURER (none) -> PCB antenna; MPN (none) -> N/A; Notes (none) -> PCB NFC loop; tune on first article.
- C183: footprint (none) -> Capacitor_SMD:C_0402_1005Metric; DISTRIBUTOR_LINK (none) -> https://www.mouser.com/ProductDetail/Murata-Electronics/GRM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; MANUFACTURER (none) -> Murata; MPN (none) -> GRM155R71A224KE01D; Notes (none) -> N/A
- C184, C187, C192, C195, C196, C203: footprint (none) -> Capacitor_SMD:C_0402_1005Metric; DISTRIBUTOR_LINK (none) -> https://www.mouser.com/ProductDetail/Murata-Electronics/GRM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; MANUFACTURER (none) -> Murata; MPN (none) -> GRM155R71C104KA88D; Notes (none) -> N/A
- C185, C188, C191: footprint (none) -> Capacitor_SMD:C_0402_1005Metric; DISTRIBUTOR_LINK (none) -> https://eu.mouser.com/en/ProductDetail/Murata-Electronics/G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; MANUFACTURER (none) -> Murata; MPN (none) -> GRM1555C1H472JE01D; Notes (none) -> Exact Rev-A fitted C0G capacitor; no substitution without R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
- C186, C189, C190, C204: footprint (none) -> Capacitor_SMD:C_0805_2012Metric; DISTRIBUTOR_LINK (none) -> https://www.mouser.com/ProductDetail/Murata-Electronics/GRM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; MANUFACTURER (none) -> Murata; MPN (none) -> GRM21BR71A106KE51L; Notes (none) -> Verify effective capacitance under DC bias.
- C193, C211, C212, C221, C222: footprint (none) -> Capacitor_SMD:C_1206_3216Metric; DISTRIBUTOR_LINK (none) -> https://www.mouser.com/ProductDetail/Murata-Electronics/GRM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; MANUFACTURER (none) -> Murata; MPN (none) -> GRM31CR71A226KE15L; Notes (none) -> Verify effective capacitance under DC bias.
- C194, C197, C199, C201, C202: footprint (none) -> Capacitor_SMD:C_0402_1005Metric; DISTRIBUTOR_LINK (none) -> https://www.mouser.com/ProductDetail/Murata-Electronics/GJM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; MANUFACTURER (none) -> Murata; MPN (none) -> GJM1555C1H2R0BB01D; Notes (none) -> N/A
- C198, C200: footprint (none) -> Capacitor_SMD:C_0402_1005Metric; DISTRIBUTOR_LINK (none) -> N/A; MANUFACTURER (none) -> N/A; MPN (none) -> N/A; Notes (none) -> Rev-A DNP; UWB shunt-tuning position; fit only after VNA me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
- C205: footprint (none) -> Capacitor_SMD:C_0603_1608Metric; DISTRIBUTOR_LINK (none) -> https://www.mouser.com/ProductDetail/Murata-Electronics/GRM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; MANUFACTURER (none) -> Murata; MPN (none) -> GRM188R71C103KA01D; Notes (none) -> N/A
- C206, C207, C209, C210, C219, C220, C232, C237: footprint (none) -> Capacitor_SMD:C_0603_1608Metric; DISTRIBUTOR_LINK (none) -> https://www.mouser.com/ProductDetail/Murata-Electronics/GRM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; MANUFACTURER (none) -> Murata; MPN (none) -> GRM188R71C104KA01D; Notes (none) -> N/A
- C208, C226, C251, C252: footprint (none) -> Capacitor_SMD:C_0603_1608Metric; DISTRIBUTOR_LINK (none) -> https://www.mouser.com/ProductDetail/Murata-Electronics/GRM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; MANUFACTURER (none) -> Murata; MPN (none) -> GRM1885C1H102JA01D; Notes (none) -> N/A
- C213, C223: footprint (none) -> Capacitor_SMD:C_0603_1608Metric; DISTRIBUTOR_LINK (none) -> https://www.mouser.com/ProductDetail/Murata-Electronics/GRM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; MANUFACTURER (none) -> Murata; MPN (none) -> GRM1885C1H470JA01D; Notes (none) -> Rev-A DNP; LF resonance trim option; populate only after me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
- C214, C224: footprint (none) -> Capacitor_SMD:C_0603_1608Metric; DISTRIBUTOR_LINK (none) -> https://www.mouser.com/ProductDetail/Murata-Electronics/GRM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; MANUFACTURER (none) -> Murata; MPN (none) -> GRM1885C1H101JA01D; Notes (none) -> Rev-A DNP; LF resonance trim option; populate only after me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
- C215, C225: footprint (none) -> Capacitor_SMD:C_0603_1608Metric; DISTRIBUTOR_LINK (none) -> https://www.mouser.com/ProductDetail/Murata-Electronics/GRM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; MANUFACTURER (none) -> Murata; MPN (none) -> GRM1885C1H221JA01D; Notes (none) -> Rev-A DNP; LF resonance trim option; populate only after me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
- C216, C218, C227, C229: footprint (none) -> Capacitor_SMD:C_0603_1608Metric; DISTRIBUTOR_LINK (none) -> https://www.mouser.com/ProductDetail/Murata-Electronics/GRM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; MANUFACTURER (none) -> Murata; MPN (none) -> GRM1885C1H221JA01D; Notes (none) -> N/A
- C217, C228: footprint (none) -> Capacitor_SMD:C_0603_1608Metric; DISTRIBUTOR_LINK (none) -> https://www.mouser.com/ProductDetail/Murata-Electronics/GRM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; MANUFACTURER (none) -> Murata; MPN (none) -> GRM1885C1H332JA01D; Notes (none) -> N/A
- C230: footprint (none) -> Capacitor_SMD:C_0603_1608Metric; DISTRIBUTOR_LINK (none) -> https://www.mouser.com/ProductDetail/Murata-Electronics/GRM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; MANUFACTURER (none) -> Murata; MPN (none) -> GRM188R71C105KA12D; Notes (none) -> N/A
- C231, C238: footprint (none) -> Capacitor_SMD:C_0805_2012Metric; DISTRIBUTOR_LINK (none) -> https://www.mouser.com/ProductDetail/Murata-Electronics/GRM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; MANUFACTURER (none) -> Murata; MPN (none) -> GRM21BR71A475KA73L; Notes (none) -> Verify effective capacitance under DC bias.
- C233, C234, C255, C256: footprint (none) -> Capacitor_SMD:C_0603_1608Metric; DISTRIBUTOR_LINK (none) -> https://www.mouser.com/ProductDetail/Murata-Electronics/GRM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; MANUFACTURER (none) -> Murata; MPN (none) -> GRM188R71A225KE15D; Notes (none) -> N/A
- C235, C236: footprint (none) -> Capacitor_SMD:C_0603_1608Metric; DISTRIBUTOR_LINK (none) -> https://www.mouser.com/en/ProductDetail/Murata-Electronics/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; MANUFACTURER (none) -> Murata; MPN (none) -> GRM1885C1H120JA01D; Notes (none) -> Rev-A DNP; optional PN7160 low-power field-detection coupli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
- C239, C245: footprint (none) -> Capacitor_SMD:C_0603_1608Metric; DISTRIBUTOR_LINK (none) -> https://www.mouser.com/ProductDetail/Murata-Electronics/GRM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; MANUFACTURER (none) -> Murata; MPN (none) -> GRM1885C1H331JA01D; Notes (none) -> N/A
- C240, C242, C244, C246, C248, C250: footprint (none) -> Capacitor_SMD:C_0603_1608Metric; DISTRIBUTOR_LINK (none) -> N/A; MANUFACTURER (none) -> DNP; MPN (none) -> N/A; Notes (none) -> Rev-A DNP; optional NFC matching trim; fit only after anten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
- C241, C247: footprint (none) -> Capacitor_SMD:C_0603_1608Metric; DISTRIBUTOR_LINK (none) -> https://www.mouser.com/ProductDetail/Murata-Electronics/GRM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; MANUFACTURER (none) -> Murata; MPN (none) -> GRM1885C1H680JA01D; Notes (none) -> N/A
- C243, C249: footprint (none) -> Capacitor_SMD:C_0603_1608Metric; DISTRIBUTOR_LINK (none) -> https://www.mouser.com/ProductDetail/Murata-Electronics/GRM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; MANUFACTURER (none) -> Murata; MPN (none) -> GRM1885C1H101JA01D; Notes (none) -> N/A
- C253, C254: footprint (none) -> Capacitor_SMD:C_0603_1608Metric; DISTRIBUTOR_LINK (none) -> https://www.mouser.com/ProductDetail/Murata-Electronics/GRM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; MANUFACTURER (none) -> Murata; MPN (none) -> GRM1885C1H150JA01D; Notes (none) -> N/A
- FB8: value BLM15AG601SN1D -> BLM15PX330SN1D; footprint (none) -> Inductor_SMD:L_0402_1005Metric; DISTRIBUTOR_LINK (none) -> https://www.mouser.com/ProductDetail/Murata-Electronics/BLM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; MANUFACTURER (none) -> Murata; MPN (none) -> BLM15PX330SN1D; Notes (none) -> 33 Ω @ 100 MHz
- J13: value Conn_Coaxial -> U.FL-R-SMT-1(10); DISTRIBUTOR_LINK (none) -> https://www.mouser.com/ProductDetail/Hirose-Connector/U.FL-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; MANUFACTURER (none) -> Hirose; MPN (none) -> U.FL-R-SMT-1(10); Notes (none) -> Inspect center-contact soldering.
- L33: footprint (none) -> Inductor_SMD:L_0402_1005Metric; DISTRIBUTOR_LINK (none) -> https://www.mouser.com/ProductDetail/Murata-Electronics/LQG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; MANUFACTURER (none) -> Murata; MPN (none) -> LQG15HS27NJ02D; Notes (none) -> N/A
- L34, L35: footprint (none) -> Inductor_SMD:L_0603_1608Metric; DISTRIBUTOR_LINK (none) -> https://www.mouser.com/ProductDetail/Murata-Electronics/LQW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; MANUFACTURER (none) -> Murata; MPN (none) -> LQW18ANR16G00D; Notes (none) -> Confirm value after NFC antenna tuning.
- L38, L39: DISTRIBUTOR_LINK (none) -> N/A; MANUFACTURER (none) -> Custom; MPN (none) -> CUSTOM-LF-COIL-134K2-REV-A; Notes (none) -> Procurement hold—final coil after enclosure/VNA measurement
- R114, R115, R116, R117: footprint (none) -> Resistor_SMD:R_0603_1608Metric; DISTRIBUTOR_LINK (none) -> https://www.mouser.com/ProductDetail/YAGEO/RC0603JR-070RL?q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; MANUFACTURER (none) -> Yageo; MPN (none) -> RC0603JR-070RL; Notes (none) -> N/A
- R118: footprint (none) -> Resistor_SMD:R_0603_1608Metric; DISTRIBUTOR_LINK (none) -> https://www.mouser.com/ProductDetail/YAGEO/RC0603FR-0710RL?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; MANUFACTURER (none) -> Yageo; MPN (none) -> RC0603FR-0710RL; Notes (none) -> N/A
- R119: footprint (none) -> Resistor_SMD:R_0603_1608Metric; DISTRIBUTOR_LINK (none) -> https://www.mouser.com/ProductDetail/YAGEO/RC0603FR-0710KL?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; MANUFACTURER (none) -> Yageo; MPN (none) -> RC0603FR-0710KL; Notes (none) -> N/A
- R120: footprint (none) -> Resistor_SMD:R_0603_1608Metric; DISTRIBUTOR_LINK (none) -> https://www.mouser.com/ProductDetail/YAGEO/RC0603FR-07100KL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; MANUFACTURER (none) -> Yageo; MPN (none) -> RC0603FR-07100KL; Notes (none) -> N/A
- R121, R122: footprint (none) -> Resistor_SMD:R_0603_1608Metric; DISTRIBUTOR_LINK (none) -> https://www.mouser.com/ProductDetail/Yageo/RC0603FR-071KL?q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; MANUFACTURER (none) -> Yageo; MPN (none) -> RC0603FR-071KL; Notes (none) -> N/A
- R123, R128: footprint (none) -> Resistor_SMD:R_0603_1608Metric; DISTRIBUTOR_LINK (none) -> https://www.mouser.com/ProductDetail/YAGEO/RC0603FR-07220RL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; MANUFACTURER (none) -> Yageo; MPN (none) -> RC0603FR-07220RL; Notes (none) -> N/A
- R124, R127, R129, R132: footprint (none) -> Resistor_SMD:R_0805_2012Metric; DISTRIBUTOR_LINK (none) -> https://www.mouser.com/ProductDetail/Panasonic/ERJ-P06J4R7V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; MANUFACTURER (none) -> Panasonic; MPN (none) -> ERJ-P06J4R7V; Notes (none) -> N/A
- R125, R130: footprint (none) -> Resistor_SMD:R_0603_1608Metric; DISTRIBUTOR_LINK (none) -> https://www.mouser.com/ProductDetail/YAGEO/RC0603FR-07150KL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; MANUFACTURER (none) -> Yageo; MPN (none) -> RC0603FR-07150KL; Notes (none) -> N/A
- R126, R131: footprint (none) -> Resistor_SMD:R_0603_1608Metric; DISTRIBUTOR_LINK (none) -> https://www.mouser.com/ProductDetail/YAGEO/RC0603FR-0747KL?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; MANUFACTURER (none) -> Yageo; MPN (none) -> RC0603FR-0747KL; Notes (none) -> N/A
- R133, R134: footprint (none) -> Resistor_SMD:R_0603_1608Metric; DISTRIBUTOR_LINK (none) -> https://www.mouser.com/ProductDetail/YAGEO/RC0603FR-072K2L?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; MANUFACTURER (none) -> Yageo; MPN (none) -> RC0603FR-072K2L; Notes (none) -> N/A
- R135, R136: footprint (none) -> Resistor_SMD:R_0805_2012Metric; DISTRIBUTOR_LINK (none) -> https://www.mouser.com/ProductDetail/Panasonic/ERJ-P06J2R7V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; MANUFACTURER (none) -> Panasonic; MPN (none) -> ERJ-P06J2R7V; Notes (none) -> N/A
- R137: footprint (none) -> Resistor_SMD:R_0603_1608Metric; DISTRIBUTOR_LINK (none) -> https://www.mouser.com/ProductDetail/YAGEO/RC0603FR-076K8L?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; MANUFACTURER (none) -> Yageo; MPN (none) -> RC0603FR-076K8L; now fitted
- R138: footprint (none) -> Resistor_SMD:R_0603_1608Metric; DISTRIBUTOR_LINK (none) -> https://www.mouser.com/ProductDetail/YAGEO/RC0603FR-076K8L?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; MANUFACTURER (none) -> Yageo; MPN (none) -> RC0603FR-076K8L; Notes (none) -> N/A; now fitted
- U35: DISTRIBUTOR_LINK (none) -> https://www.mouser.com/ProductDetail/Qorvo/DW3220TR13?qs=hW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; MANUFACTURER (none) -> Qorvo; MPN (none) -> DW3220TR13; Notes (none) -> N/A
- U41: DISTRIBUTOR_LINK (none) -> https://www.mouser.com/ProductDetail/u-blox/MAX-M10N-10B?qs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; MANUFACTURER (none) -> u-blox; MPN (none) -> MAX-M10N-10B-00; Notes (none) -> N/A
- U44: value PN7160B1HN/C101Y -> PN7160B1HN/C100E; DISTRIBUTOR_LINK (none) -> https://www.digikey.com/en/products/detail/nxp-usa-inc/PN71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; MANUFACTURER (none) -> NXP; MPN (none) -> PN7160B1HN/C100E; Notes (none) -> N/A
- U45, U46: DISTRIBUTOR_LINK (none) -> https://www.mouser.com/ProductDetail/Texas-Instruments/TMS3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; MANUFACTURER (none) -> Texas Instruments; MPN (none) -> TMS3705FDRQ1; Notes (none) -> SOURCING: recheck lifecycle and stock before PO.
- U47: DISTRIBUTOR_LINK (none) -> https://www.digikey.co.uk/en/products/detail/texas-instrume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; MANUFACTURER (none) -> Texas Instruments; MPN (none) -> SN74AHCT00PWR; Notes (none) -> N/A
- U48: DISTRIBUTOR_LINK (none) -> https://www.mouser.com/ProductDetail/Texas-Instruments/SN74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; MANUFACTURER (none) -> Texas Instruments; MPN (none) -> SN74LVC157APWR; Notes (none) -> N/A
- Y10, Y9: DISTRIBUTOR_LINK (none) -> https://www.mouser.com/ProductDetail/Murata-Electronics/CST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; MPN (none) -> CSTCR4M00G55B-R0; Notes (none) -> N/A
- Y7: DISTRIBUTOR_LINK (none) -> https://www.digikey.co.uk/en/products/detail/txc-corporatio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; MANUFACTURER (none) -> TXC; MPN (none) -> 8Y38472012; Notes (none) -> Verify crystal load capacitance.
- Y8: value NX2016SA 27.12MHz EXS00A-CS06346 -> NX2016SA 27.12MHz 10pF; footprint (none) -> Crystal:Crystal_SMD_2016-4Pin_2.0x1.6mm; DISTRIBUTOR_LINK (none) -> https://www.digikey.co.uk/en/products/detail/ndk-nihon-demp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; MANUFACTURER (none) -> NDK; MPN (none) -> NX2016SA-27.120000MHz-EXS00A-CS06346; Notes (none) -> Ground crystal case pads 2/4.
Connections:
- net UWB_VDD2B is gone; now on net +3V3: C187.1, C188.1, C189.1, U35.23 (VDD2b)
- net +3V3: now also FB8.1, R145.1, R148.2; no longer FB8.2
- net GND: now also C257.2, C258.2, R140.1, R146.2, R147.2
- net LF_A_DRV: now also J15.1 (Pin_1)
- net LF_A_TUNE: now also J15.2 (Pin_2)
- net LF_B_DRV: now also J16.1 (Pin_1)
- net LF_B_TUNE: now also J16.2 (Pin_2)
- net NFC_DWL_REQ: now also R146.1
- net NFC_VEN: now also R147.1
- net UWB_ANT1_PORT: now also AE1.1 (RF), R142.1
- net UWB_ANT2_PORT: now also AE2.1 (RF), R143.1
- net UWB_IRQ: now also R140.2
- net UWB_RF1_MATCH: now also C257.1
- net UWB_RF2_MATCH: now also C258.1
- net UWB_RST: now also R144.2; no longer U35.33 (~{RST})
- net UWB_VDD2A: now also FB8.2; no longer FB8.1
- net nCS_NFC: now also R145.2
- net nCS_UWB: now also R148.1
- new net UWB_ANT1_FTE: AE1.3 (FTE), R142.2
- new net UWB_ANT2_FTE: AE2.3 (FTE), R143.2
- new net UWB_RST_IC: R144.1, U35.33 (~{RST})
- no-connect marks 26 -> 35
Other:
- note added: "OFF-BOARD 134.2 kHz ORTHOGONAL LF COILS"
- note added: "UWB PDoA ANTENNA LAYOUT: Place AE1 and AE2 on the same PCB edge with identical orientation. Follow the Taoglas UWA.01 land pattern and maintain its 7.5 × 6.0 mm all-layer copper keepout for each antenna. Route RF1 and RF2 as phase-matched 50 Ω traces with identical transitions and grounding. Target antenna phase-centre spacing: 20.8 mm for channel 5 or 16.9 mm for channel 9 (0.45λ). Confirm the p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"
- moved on the sheet: C197, R114

Commit message: the schematic is finished
Parts:
- R137: Notes (none) -> N/A
- R144: Notes DW3220 IRQ pull-down. -> DW3220 reset series resistor.
- R145: Notes DW3220 IRQ pull-down. -> 10k pull-up on nCS_NFC.
- R146: Notes DW3220 IRQ pull-down. -> 10k pull-down on NFC_DWL_REQ.
- R147: Notes DW3220 IRQ pull-down. -> 10k pull-down on NFC_VEN.
- R148: Notes DW3220 IRQ pull-down. -> 10k pull-up on nCS_UWB.
Changed lines of the file:
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@@
 			)
 		)
-		(property "Datasheet" "https://yageogroup.com/component-documentation/download/specsheet/RC0603FR-07100KL"
+		(property "Datasheet" "https://www.yageo.com/upload/media/product/productsearch/datasheet/rchip/PYu-RC_Group_51_RoHS_L_11.pdf"
 			(at 60.96 85.09 0)
 			(hide yes)
@@
 			)
 		)
-		(property "Notes" "DW3220 IRQ pull-down."
+		(property "Notes" "DW3220 reset series resistor."
 			(at 60.96 85.09 90)
 			(hide yes)
@@
 			)
 		)
-		(property "Datasheet" "https://www.mouser.com/catalog/specsheets/JST_B4B_PH_SM4_TB_LF_SN_ePH.pdf?_gl=1*1bm4zi6*_gcl_au*MzA0ODk5NjM2LjE3ODc5Njk1Njg.*_ga*NDk1ODc5OTUzLjE3ODc5Njk1Njg.*_ga_15W4STQT4T*czE3ODgzMzYxMDQkbzE5JGcxJHQxNzg4MzM2MTA4JGo1NiRsMCRoMA.."
+		(property "Datasheet" "https://www.jst-mfg.com/product/pdf/eng/ePH.pdf"
 			(at 127 375.92 0)
 			(hide yes)
@@
 			)
 		)
-		(property "Datasheet" "https://www.mouser.com/catalog/specsheets/JST_B4B_PH_SM4_TB_LF_SN_ePH.pdf?_gl=1*1bm4zi6*_gcl_au*MzA0ODk5NjM2LjE3ODc5Njk1Njg.*_ga*NDk1ODc5OTUzLjE3ODc5Njk1Njg.*_ga_15W4STQT4T*czE3ODgzMzYxMDQkbzE5JGcxJHQxNzg4MzM2MTA4JGo1NiRsMCRoMA.."
+		(property "Datasheet" "https://www.jst-mfg.com/product/pdf/eng/ePH.pdf"
 			(at 127 363.22 0)
 			(hide yes)
@@
 			)
 		)
-		(property "Notes" "DW3220 IRQ pull-down."
+		(property "Notes" "10k pull-down on NFC_VEN."
 			(at 256.54 86.36 90)
 			(hide yes)
@@
 			)
 		)
-		(property "Notes" "DW3220 IRQ pull-down."
+		(property "Notes" "10k pull-up on nCS_NFC."
 			(at 240.03 41.91 90)
 			(hide yes)
@@
 			)
 		)
-		(property "Notes" "DW3220 IRQ pull-down."
+		(property "Notes" "10k pull-up on nCS_UWB."
 			(at 24.13 64.77 90)
 			(hide yes)
@@
 			)
 		)
-		(property "Notes" "DW3220 IRQ pull-down."
+		(property "Notes" "10k pull-down on NFC_DWL_REQ."
 			(at 246.38 86.36 90)
 			(hide yes)
@@
 			)
 		)
-		(property "Notes" ""
+		(property "Notes" "N/A"
 			(at 405.13 109.22 90)
 			(hide yes)

Commit message: finished schematic phase
Parts:
- AE1, AE2: footprint (none) -> FOBtool_Custom:Antenna_Taoglas_UWA01_3.2x1.6mm
Changed lines of the file:
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@@
 			)
 		)
-		(property "Footprint" ""
+		(property "Footprint" "FOBtool_Custom:Antenna_Taoglas_UWA01_3.2x1.6mm"
 			(at 152.4 113.03 0)
 			(hide yes)
@@
 			)
 		)
-		(property "Footprint" ""
+		(property "Footprint" "FOBtool_Custom:Antenna_Taoglas_UWA01_3.2x1.6mm"
 			(at 213.36 111.76 0)
 			(hide yes)

Commit message: adding 3d models
Parts:
- J15, J16: symbol Connector_Generic:Conn_01x02 -> FOBtool_Custom:JST_PH_2Pin_MP
Connections:
- no-connect marks 35 -> 37
Changed lines of the file:
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@@
 	)
 	(no_connect
+		(at 132.08 378.46)
+	)
+	(no_connect
 		(at 49.53 172.72)
 	)
@@
 	)
 	(no_connect
+		(at 132.08 365.76)
+	)
+	(no_connect
 		(at 74.93 236.22)
 	)
@@
 	)
 	(symbol
-		(lib_id "Connector_Generic:Conn_01x02")
+		(lib_id "FOBtool_Custom:JST_PH_2Pin_MP")
 		(at 127 375.92 0)
 		(unit 1)
@@
 		(fields_autoplaced yes)
 		(property "Reference" "J16"
-			(at 129.54 375.9199 0)
+			(at 127 369.57 0)
 			(show_name no)
 			(do_not_autoplace no)
@@
 					(size 1.27 1.27)
 				)
-				(justify left)
 			)
 		)
 		(property "Value" "S2B-PH-SM4-TB(LF)(SN)"
-			(at 129.54 378.4599 0)
+			(at 127 372.11 0)
 			(show_name no)
 			(do_not_autoplace no)
@@
 					(size 1.27 1.27)
 				)
-				(justify left)
 			)
 		)
@@
 		(pin "1"
 		)
+		(pin "MP"
+		)
 		(instances
 			(project "FOBtool_HW"
@@
 	)
 	(symbol
-		(lib_id "Connector_Generic:Conn_01x02")
+		(lib_id "FOBtool_Custom:JST_PH_2Pin_MP")
 		(at 127 363.22 0)
 		(unit 1)
@@
 		(in_pos_files yes)
 		(dnp no)
-		(fields_autoplaced yes)
 		(property "Reference" "J15"
-			(at 129.54 363.2199 0)
+			(at 127.508 360.68 0)
 			(show_name no)
 			(do_not_autoplace no)
@@
 		)
 		(property "Value" "S2B-PH-SM4-TB(LF)(SN)"
-			(at 129.54 365.7599 0)
+			(at 128.016 367.538 0)
 			(show_name no)
 			(do_not_autoplace no)
@@
 		(pin "1"
 		)
+		(pin "MP"
+		)
 		(instances

Commit message: nearly finishing placement phase
Parts:
- added J21: 781710002, Connector_Molex:Molex_Pico-EZmate_78171-0002_1x02-1MP_P1.20mm_Vertical, symbol FOBtool_Custom:JST_PH_2Pin_MP
- AE3: Notes PCB NFC loop; tune on first article. -> - External rear NFC antenna assembly—geometry, ferrite and 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
Connections:
- net NFC_ANT_LOOP_N: now also J21.2 (Pin_2)
- net NFC_ANT_LOOP_P: now also J21.1 (Pin_1)
- no-connect marks 37 -> 38
Other:
- note added: "External rear NFC antenna assembly—geometry and tuning pending"
Changed lines of the file:
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@@
 		)
 	)
+	(text "External rear NFC antenna assembly—geometry and tuning pending"
+		(exclude_from_sim no)
+		(at 385.572 132.334 0)
+		(effects
+			(font
+				(size 1.27 1.27)
+			)
+		)
+	)
 	(text "UWB TRANSCEIVER, CLOCK, DUAL ANTENNAS AND SPI"
 		(exclude_from_sim no)
@@
 	)
 	(no_connect
+		(at 400.05 147.32)
+	)
+	(no_connect
 		(at 74.93 241.3)
 	)
@@
 	(wire
 		(pts
+			(xy 370.84 147.32) (xy 389.89 147.32)
+		)
+		(stroke
+			(width 0)
+			(type default)
+		)
+	)
+	(wire
+		(pts
 			(xy 367.03 88.9) (xy 378.46 88.9)
 		)
@@
 	(wire
 		(pts
+			(xy 370.84 144.78) (xy 389.89 144.78)
+		)
+		(stroke
+			(width 0)
+			(type default)
+		)
+	)
+	(wire
+		(pts
 			(xy 256.54 80.01) (xy 289.56 80.01)
 		)
@@
 		)
 	)
+	(label "NFC_ANT_LOOP_N"
+		(at 370.84 147.32 0)
+		(effects
+			(font
+				(size 1.27 1.27)
+			)
+			(justify left bottom)
+		)
+	)
 	(label "NFC_RX_MATCH_N"
 		(at 383.54 118.11 0)
@@
 		)
 	)
+	(label "NFC_ANT_LOOP_P"
+		(at 370.84 144.78 0)
+		(effects
+			(font
+				(size 1.27 1.27)
+			)
+			(justify left bottom)
+		)
+	)
 	(label "LF_B_RETURN"
 		(at 313.69 269.24 180)
@@
 	)
 	(symbol
+		(lib_id "FOBtool_Custom:JST_PH_2Pin_MP")
+		(at 394.97 144.78 0)
+		(unit 1)
+		(body_style 1)
+		(exclude_from_sim no)
+		(in_bom yes)
+		(on_board yes)
+		(in_pos_files yes)
+		(dnp no)
+		(property "Reference" "J21"
+			(at 395.478 142.24 0)
+			(show_name no)
+			(do_not_autoplace no)
+			(effects
+				(font
+					(size 1.27 1.27)
+				)
+				(justify left)
+			)
+		)
+		(property "Value" "781710002"
+			(at 395.986 149.098 0)
+			(show_name no)
+			(do_not_autoplace no)
+			(effects
+				(font
+					(size 1.27 1.27)
+				)
+				(justify left)
+			)
+		)
+		(property "Footprint" "Connector_Molex:Molex_Pico-EZmate_78171-0002_1x02-1MP_P1.20mm_Vertical"
+			(at 394.97 144.78 0)
+			(hide yes)
+			(show_name no)
+			(do_not_autoplace no)
+			(effects
+				(font
+					(size 1.27 1.27)
+				)
+			)
+		)
+		(property "Datasheet" "https://www.molex.com/en-us/products/part-detail/781710002?display=pdf&utm_source=M2X&utm_medium=api&utm_campaign=api&utm_id=M2X_API?utm_source=M2X&utm_medium=api&utm_campaign=api&utm_id=M2X_API"
+			(at 394.97 144.78 0)
+			(hide yes)
+			(show_name no)
+			(do_not_autoplace no)
+			(effects
+				(font
+					(size 1.27 1.27)
+				)
+			)
+		)
+		(property "Description" "Generic connector, single row, 01x02, script generated (kicad-library-utils/schlib/autogen/connector/)"
+			(at 394.97 144.78 0)
+			(hide yes)
+			(show_name no)
+			(do_not_autoplace no)
+			(effects
+				(font
+					(size 1.27 1.27)
+				)
+			)
+		)
+		(property "DISTRIBUTOR_LINK" "https://eu.mouser.com/en/ProductDetail/Molex/78171-0002?qs=Gs2o0dzr3RhBbmnwhRVwhg%3D%3D&srsltid=AU7gw4WN5d6vVQCp-ntq4lPJklX13r7iXxG4NABma2jFhMtAI4v6GnZP"
+			(at 394.97 144.78 0)
+			(hide yes)
+			(show_name no)
+			(do_not_autoplace no)
+			(effects
+				(font
+					(size 1.27 1.27)
+				)
+			)
+		)
+		(property "MANUFACTURER" "Molex"
+			(at 394.97 144.78 0)
+			(hide yes)
+			(show_name no)
+			(do_not_autoplace no)
+			(effects
+				(font
+					(size 1.27 1.27)
+				)
+			)
+		)
+		(property "MPN" "781710002"
+			(at 394.97 144.78 0)
+			(hide yes)
+			(show_name no)
+			(do_not_autoplace no)
+			(effects
+				(font
+					(size 1.27 1.27)
+				)
+			)
+		)
+		(property "Notes" "External NFC antenna connection. Pin 1=NFC_ANT_LOOP_P; pin 2=NFC_ANT_LOOP_N."
+			(at 394.97 144.78 0)
+			(hide yes)
+			(show_name no)
+			(do_not_autoplace no)
+			(effects
+				(font
+					(size 1.27 1.27)
+				)
+			)
+		)
+		(pin "2"
+		)
+		(pin "1"
+		)
+		(pin "MP"
+		)
+		(instances
+			(project "FOBtool_HW"
+				(path "/4178b7d0-cf29-4cf2-b214-acbbbd97d338/e68072eb-1a73-49dc-9cee-ac0e0ab7a67a"
+					(reference "J21")
+					(unit 1)
+				)
+			)
+		)
+	)
+	(symbol
 		(lib_id "power:GND")
 		(at 189.23 104.14 0)
@@
 		(exclude_from_sim no)
 		(in_bom yes)
-		(on_board yes)
-		(in_pos_files yes)
+		(on_board no)
+		(in_pos_files no)
 		(dnp no)
 		(fields_autoplaced yes)
@@
 			)
 		)
-		(property "Notes" "PCB NFC loop; tune on first article."
+		(property "Notes" "- External rear NFC antenna assembly—geometry, ferrite and tuning pending."
 			(at 374.65 124.46 90)
 			(hide yes)
